File: boxes/ics/NB3_hindbrain/NB3_hindbrain.kicad_sch (KiCad schematic)
At the start: 56 parts, among them IC1 FPGA_ICE40UP5K-SG48I, IC2 NOR_Flash_W25Q32JVSSIQ, J1 MicroUSB_10103594-0001LF, J2 Conn_01x20_Male, J3 Conn_01x20_Male, U1 EEPROM_93LC56BT-I-OT, Y1 Osc_12MHz_ECS-2520MV-120-BN-TR

Commit message: Update KiCAD for NB3 hindbrain
Parts:
- added U2: USBtoSPI_FT4232HL, NB3_hindbrain:USBtoSPI_FT4232HL, symbol NB3_hindbrain:USBtoSPI_FT4232HL
Connections:
- net +1V8: now also U2.12 (VCORE), U2.37 (VCORE), U2.49 (VREGOUT), U2.64 (VCORE)
- net +3V3: now also U2.20 (VCCIO), U2.31 (VCCIO), U2.42 (VCCIO); no longer FB1.2, FB2.2
- net CDONE: now also U2.19 (ADBUS3), U2.29 (BDBUS3)
- net CLK_12MHz: now also U2.2 (OSCI)
- net CRESET_B: now also U2.21 (ADBUS4), U2.30 (BDBUS4)
- net EECS: now also U2.33 (BDBUS6)
- net EEDATA_I: now also U2.34 (BDBUS7)
- net FLASH_HOLDn: now also U2.28 (BDBUS2)
- net FLASH_SCK: now also U2.22 (ADBUS5), U2.8 (DP)
- net FLASH_SI: now also U2.24 (ADBUS7), U2.63 (EECS)
- net FLASH_SO: now also U2.23 (ADBUS6), U2.61 (EEDATA)
- net FLASH_SSn: now also U2.17 (ADBUS1), U2.27 (BDBUS1)
- net FT_VPHY: now also U2.4 (VPHY)
- net FT_VPLL: now also U2.9 (VPLL)
- net GND: now also U2.1 (GND), U2.10 (AGND), U2.11 (GND), U2.15 (GND), U2.25 (GND), U2.35 (GND), U2.47 (GND), U2.5 (GND), U2.51 (GND)
- net at R7.2: now also U2.6 (REF)
- new net: FB1.2, FB2.2, U2.50 (VREGIN), U2.56 (VCCIO)

Commit message: Update NB3 PCBs and parts
Parts:
- removed U2: USBtoSPI_FT4232HL, NB3_hindbrain:USBtoSPI_FT4232HL, symbol NB3_hindbrain:USBtoSPI_FT4232HL
- added IC3: FT232HL, QFP50P900X900X160-48N, symbol NB3_hindbrain:USBtoSPI_FT232HL
Changed lines of the file:
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@@
   (junction (at 100.33 140.97) (diameter 0.9144) (color 0 0 0 0)
   )
-  (junction (at 99.06 17.78) (diameter 0.9144) (color 0 0 0 0)
-  )
   (junction (at 19.05 38.1) (diameter 0.9144) (color 0 0 0 0)
   )
@@
   (junction (at 25.4 156.21) (diameter 0.9144) (color 0 0 0 0)
   )
-  (junction (at 88.9 114.3) (diameter 0) (color 0 0 0 0)
-  )
   (junction (at 140.97 161.925) (diameter 0.9144) (color 0 0 0 0)
   )
@@
   (junction (at 19.05 45.72) (diameter 0.9144) (color 0 0 0 0)
   )
-  (junction (at 104.14 114.3) (diameter 0) (color 0 0 0 0)
-  )
   (junction (at 19.05 48.26) (diameter 0.9144) (color 0 0 0 0)
   )
@@
   (junction (at 190.5 134.62) (diameter 0.9144) (color 0 0 0 0)
   )
-  (junction (at 106.68 114.3) (diameter 0) (color 0 0 0 0)
-  )
-  (junction (at 96.52 17.78) (diameter 0) (color 0 0 0 0)
-  )
   (junction (at 198.12 134.62) (diameter 0.9144) (color 0 0 0 0)
   )
@@
   (junction (at 87.63 161.925) (diameter 0.9144) (color 0 0 0 0)
   )
-  (junction (at 101.6 114.3) (diameter 0) (color 0 0 0 0)
-  )
   (junction (at 37.465 79.375) (diameter 0.9144) (color 0 0 0 0)
   )
-  (junction (at 91.44 114.3) (diameter 0) (color 0 0 0 0)
-  )
   (junction (at 21.59 88.9) (diameter 0.9144) (color 0 0 0 0)
   )
   (junction (at 217.17 67.31) (diameter 0.9144) (color 0 0 0 0)
   )
-  (junction (at 96.52 114.3) (diameter 0) (color 0 0 0 0)
-  )
   (junction (at 19.05 35.56) (diameter 0.9144) (color 0 0 0 0)
   )
@@
   (junction (at 111.76 140.97) (diameter 0.9144) (color 0 0 0 0)
   )
-  (junction (at 99.06 114.3) (diameter 0) (color 0 0 0 0)
-  )
   (junction (at 193.04 107.95) (diameter 0.9144) (color 0 0 0 0)
   )
@@
     (stroke (width 0) (type solid))
   )
-  (wire (pts (xy 91.44 114.3) (xy 93.98 114.3))
-    (stroke (width 0) (type solid))
-  )
   (wire (pts (xy 217.17 67.31) (xy 217.17 72.39))
     (stroke (width 0) (type solid))
@@
     (stroke (width 0) (type solid))
   )
-  (wire (pts (xy 101.6 114.3) (xy 104.14 114.3))
-    (stroke (width 0) (type solid))
-  )
   (wire (pts (xy 133.35 25.4) (xy 134.62 25.4))
     (stroke (width 0) (type solid))
@@
     (stroke (width 0) (type solid))
   )
-  (wire (pts (xy 96.52 114.3) (xy 99.06 114.3))
-    (stroke (width 0) (type solid))
-  )
   (polyline (pts (xy 12.7 22.86) (xy 55.88 22.86))
     (stroke (width 0) (type dash))
@@
     (stroke (width 0) (type solid))
   )
-  (wire (pts (xy 83.82 114.3) (xy 88.9 114.3))
+  (wire (pts (xy 83.82 114.3) (xy 93.98 114.3))
     (stroke (width 0) (type solid))
   )
@@
     (stroke (width 0) (type solid))
   )
-  (wire (pts (xy 104.14 114.3) (xy 106.68 114.3))
+  (wire (pts (xy 93.98 114.3) (xy 114.3 114.3))
     (stroke (width 0) (type solid))
   )
@@
     (stroke (width 0) (type solid))
   )
-  (wire (pts (xy 96.52 17.78) (xy 99.06 17.78))
+  (wire (pts (xy 93.98 17.78) (xy 99.06 17.78))
     (stroke (width 0) (type solid))
   )
@@
     (stroke (width 0) (type solid))
   )
-  (wire (pts (xy 88.9 114.3) (xy 91.44 114.3))
-    (stroke (width 0) (type solid))
-  )
   (wire (pts (xy 33.655 177.165) (xy 37.465 177.165))
     (stroke (width 0) (type solid))
@@
     (stroke (width 0) (type solid))
   )
-  (wire (pts (xy 99.06 114.3) (xy 101.6 114.3))
-    (stroke (width 0) (type solid))
-  )
   (wire (pts (xy 209.55 151.13) (xy 219.71 151.13))
     (stroke (width 0) (type solid))
@@
     (stroke (width 0) (type solid))
   )
-  (wire (pts (xy 93.98 114.3) (xy 96.52 114.3))
-    (stroke (width 0) (type solid))
-  )
   (wire (pts (xy 47.625 74.93) (xy 47.625 79.375))
     (stroke (width 0) (type solid))
@@
     (stroke (width 0) (type solid))
   )
-  (wire (pts (xy 93.98 17.78) (xy 96.52 17.78))
-    (stroke (width 0) (type solid))
-  )
   (wire (pts (xy 21.59 106.68) (xy 68.58 106.68))
     (stroke (width 0) (type solid))
@@
     (stroke (width 0) (type solid))
   )
-  (wire (pts (xy 99.06 17.78) (xy 99.06 17.78))
-    (stroke (width 0) (type solid))
-  )
   (wire (pts (xy 205.74 67.31) (xy 217.17 67.31))
     (stroke (width 0) (type solid))
@@
     (stroke (width 0) (type solid))
   )
-  (wire (pts (xy 106.68 114.3) (xy 114.3 114.3))
-    (stroke (width 0) (type solid))
-  )
   (wire (pts (xy 148.59 169.545) (xy 162.56 169.545))
     (stroke (width 0) (type solid))
@@
     )
   )
-  (symbol (lib_id "NB3_hindbrain:USBtoSPI_FT4232HL") (at 73.66 22.86 0) (unit 1)
-    (in_bom yes) (on_board yes) (dnp no) (fields_autoplaced)
-    (property "Reference" "U2" (at 103.4289 19.3308 0)
-      (effects (font (size 1.27 1.27)) (justify left))
-    )
-    (property "Value" "USBtoSPI_FT4232HL" (at 103.4289 21.3788 0)
-      (effects (font (size 1.27 1.27)) (justify left))
-    )
-    (property "Footprint" "NB3_hindbrain:USBtoSPI_FT4232HL" (at 73.66 132.08 0)
-      (effects (font (size 1.27 1.27)) (justify left bottom) hide)
-    )
-    (property "Datasheet" "" (at 73.66 129.54 0)
-      (effects (font (size 1.27 1.27)) (justify left bottom) hide)
-    )
-    (property "DESCRIPTION" "USB Hi-Speed to Quad Channel Serial UART/JTAG/SPI/I2C IC - LQFP-64" (at 73.66 127 0)
-      (effects (font (size 1.27 1.27)) (justify left bottom) hide)
-    )
-    (property "AVAILABILITY" "Unavailable" (at 73.66 139.7 0)
-      (effects (font (size 1.27 1.27)) (justify left bottom) hide)
-    )
-    (property "MP" "FT4232HL" (at 73.66 137.16 0)
-      (effects (font (size 1.27 1.27)) (justify left bottom) hide)
-    )
-    (property "PRICE" "None" (at 73.66 134.62 0)
-      (effects (font (size 1.27 1.27)) (justify left bottom) hide)
-    )
-    (property "MF" "FTDI, Future" (at 73.66 142.24 0)
-      (effects (font (size 1.27 1.27)) (justify left bottom) hide)
-    )
-    (property "PACKAGE" "LQFP-64 FTDI" (at 73.66 129.54 0)
-      (effects (font (size 1.27 1.27)) (justify left bottom) hide)
-    )
-    (pin "1")
-    (pin "10")
-    (pin "11")
-    (pin "12")
-    (pin "13")
-    (pin "14")
-    (pin "15")
-    (pin "16")
-    (pin "17")
-    (pin "18")
-    (pin "19")
-    (pin "2")
-    (pin "20")
-    (pin "21")
-    (pin "22")
-    (pin "23")
-    (pin "24")
-    (pin "25")
-    (pin "26")
-    (pin "27")
-    (pin "28")
-    (pin "29")
-    (pin "3")
-    (pin "30")
-    (pin "31")
-    (pin "32")
-    (pin "33")
-    (pin "34")
-    (pin "35")
-    (pin "36")
-    (pin "37")
-    (pin "38")
-    (pin "39")
-    (pin "4")
-    (pin "40")
-    (pin "41")
-    (pin "42")
-    (pin "43")
-    (pin "44")
-    (pin "45")
-    (pin "46")
-    (pin "47")
-    (pin "48")
-    (pin "49")
-    (pin "5")
-    (pin "50")
-    (pin "51")
-    (pin "52")
-    (pin "53")
-    (pin "54")
-    (pin "55")
-    (pin "56")
-    (pin "57")
-    (pin "58")
-    (pin "59")
-    (pin "6")
-    (pin "60")
-    (pin "61")
-    (pin "62")
-    (pin "63")
-    (pin "64")
-    (pin "7")
-    (pin "8")
-    (pin "9")
-    (instances
-      (project "NB3_hindbrain"
-        (path "/c49eb9c2-071f-42f1-813b-8f9aeee9d910"
-          (reference "U2") (unit 1)
-        )
-      )
-    )
-  )
   (symbol (lib_id "power:GND") (at 30.48 53.34 0) (unit 1)
     (in_bom yes) (on_board yes) (dnp no)
@@
         )
       )
+    )
+  )
+  (symbol (lib_id "NB3_hindbrain:USBtoSPI_FT232HL") (at 71.12 54.61 0) (unit 1)
+    (in_bom yes) (on_board yes) (dnp no) (fields_autoplaced)
+    (property "Reference" "IC3" (at 113.9481 48.8963 0)
+      (effects (font (size 1.27 1.27)))
+    )
+    (property "Value" "FT232HL" (at 113.9481 50.9443 0)
+      (effects (font (size 1.27 1.27)))
+    )
+    (property "Footprint" "QFP50P900X900X160-48N" (at 110.49 136.83 0)
+      (effects (font (size 1.27 1.27)) (justify left top) hide)
+    )
+    (property "Datasheet" "http://www.ftdichip.com/Support/Documents/DataSheets/ICs/DS_FT232H.pdf" (at 110.49 236.83 0)
+      (effects (font (size 1.27 1.27)) (justify left top) hide)
+    )
+    (property "Height" "1.6" (at 110.49 436.83 0)
+      (effects (font (size 1.27 1.27)) (justify left top) hide)
+    )
+    (property "Mouser Part Number" "895-FT232HL-REEL" (at 110.49 536.83 0)
+      (effects (font (size 1.27 1.27)) (justify left top) hide)
+    )
+    (property "Mouser Price/Stock" "https://www.mouser.co.uk/ProductDetail/FTDI/FT232HL-REEL?qs=rzPzygjq8vIanTFlYsBQCw%3D%3D" (at 110.49 636.83 0)
+      (effects (font (size 1.27 1.27)) (justify left top) hide)
+    )
+    (property "Manufacturer_Name" "FTDI Chip" (at 110.49 736.83 0)
+      (effects (font (size 1.27 1.27)) (justify left top) hide)
+    )
+    (property "Manufacturer_Part_Number" "FT232HL-REEL" (at 110.49 836.83 0)
+      (effects (font (size 1.27 1.27)) (justify left top) hide)
+    )
+    (pin "1")
+    (pin "10")
+    (pin "11")
+    (pin "12")
+    (pin "13")
+    (pin "14")
+    (pin "15")
+    (pin "16")
+    (pin "17")
+    (pin "18")
+    (pin "19")
+    (pin "2")
+    (pin "20")
+    (pin "21")
+    (pin "22")
+    (pin "23")
+    (pin "24")
+    (pin "25")
+    (pin "26")
+    (pin "27")
+    (pin "28")
+    (pin "29")
+    (pin "3")
+    (pin "30")
+    (pin "31")
+    (pin "32")
+    (pin "33")
+    (pin "34")
+    (pin "35")
+    (pin "36")
+    (pin "37")
+    (pin "38")
+    (pin "39")
+    (pin "4")
+    (pin "40")
+    (pin "41")
+    (pin "42")
+    (pin "43")
+    (pin "44")
+    (pin "45")
+    (pin "46")
+    (pin "47")
+    (pin "48")
+    (pin "5")
+    (pin "6")
+    (pin "7")
+    (pin "8")
+    (pin "9")
+    (instances
+      (project "NB3_hindbrain"
+        (path "/c49eb9c2-071f-42f1-813b-8f9aeee9d910"
+          (reference "IC3") (unit 1)
+        )
+      )
