File: boxes/audio/NB3_ear/NB3_ear.kicad_pcb (KiCad board)
At the start: 2 copper layers, 20 x 18 mm, 6 parts, among them J1 Conn_02x03_Odd_Even, J2 Conn_02x03_Odd_Even

Commit message: Update NB3_Ear (R&E Only)
Connections:
- net +3V3 renamed +3.3V
Other:
- outline, holes or cut-outs redrawn
- board text added: "Education"
- board text added: "NB3 Ear Rev 0.0.2"
- board text added: "ONLY"
- board text added: "Research"
- board text removed: "NB3 Ear Rev 0.0.1"

Commit message: Upload NB3_ear "fab" v2
Changed lines of the file:
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@@
         (effects (font (size 1 1) (thickness 0.15)))
     )
-    (fp_text value "Conn_02x03_Odd_Even" (at 0 4.87 90) (layer "F.Fab")
+    (fp_text value "Conn_02x03_Odd_Even" (at 0 4.87 90) (layer "F.Fab") hide
         (effects (font (size 1 1) (thickness 0.15)))
     )
@@
         (effects (font (size 1 1) (thickness 0.15)))
     )
-    (fp_text value "Conn_02x03_Odd_Even" (at 0 4.87 90) (layer "F.Fab")
+    (fp_text value "Conn_02x03_Odd_Even" (at 0 4.87 90) (layer "F.Fab") hide
         (effects (font (size 1 1) (thickness 0.15)))
     )
@@
     (polygon
       (pts
-        (xy 141.58 98.775)
-        (xy 160.58 98.775)
-        (xy 160.58 115.775)
-        (xy 141.58 115.775)
+        (xy 141.842 99.003)
+        (xy 160.384 99.003)
+        (xy 160.384 115.513)
+        (xy 141.842 115.513)
       )
     )
@@
     (connect_pads (clearance 0.25))
     (min_thickness 0.254) (filled_areas_thickness no)
-    (fill (thermal_gap 0.508) (thermal_bridge_width 0.508))
+    (fill yes (thermal_gap 0.508) (thermal_bridge_width 0.508))
     (polygon
       (pts
-        (xy 160.58 115.775)
-        (xy 141.58 115.775)
-        (xy 141.58 98.775)
-        (xy 160.58 98.775)
+        (xy 160.384 115.513)
+        (xy 141.842 115.513)
+        (xy 141.842 99.003)
+        (xy 160.384 99.003)
       )
     )
