File: boxes/audio/NB3_ear/NB3_ear.kicad_sch (KiCad schematic)
At the start: 5 parts, among them J1 Conn_02x03_Odd_Even, J2 Conn_02x03_Odd_Even

Commit message: Update NB3_Ear (R&E Only)
Connections:
- net +3V3 renamed +3.3V
Other:
- note added: "For Research and Education Only"
