File: boxes/fpgas/NB3_hindbrain/NB3_hindbrain.kicad_pcb (KiCad board)
At the start: 4 copper layers, 57 x 22 mm, 58 parts, among them IC1 FPGA_ICE40UP5K-SG48I, IC2 NOR_Flash_W25Q32JVSSIQ, IC3 FT232HL, IC4 ADC_MCP3004-I-SL, J1 MicroUSB_10103594-0001LF, J2 Conn_01x20_Male, J3 Conn_01x20_Male, U1 EEPROM_93LC56BT-I-OT, Y1 Osc_12MHz_ECS-2520MV-120-BN-TR

Commit message: Brainsotmring NB3_hindbrain
Parts:
- added D10: LED, LED_SMD:LED_0402_1005Metric, F.Cu at (110.8, 77.0)
- added D11: LED, LED_SMD:LED_0402_1005Metric, F.Cu at (112.1, 77.0)
- added D12: LED, LED_SMD:LED_0402_1005Metric, F.Cu at (113.3, 77.0)
- added D13: LED, LED_SMD:LED_0402_1005Metric, F.Cu at (114.6, 77.0)
- added D14: LED, LED_SMD:LED_0402_1005Metric, F.Cu at (115.8, 77.0)
- added D15: LED, LED_SMD:LED_0402_1005Metric, F.Cu at (117.1, 77.0)
- added D16: LED, LED_SMD:LED_0402_1005Metric, F.Cu at (118.3, 77.0)
- added D17: LED, LED_SMD:LED_0402_1005Metric, F.Cu at (119.6, 77.0)
- added D18: LED, LED_SMD:LED_0402_1005Metric, F.Cu at (120.8, 77.0)
- added D19: LED, LED_SMD:LED_0402_1005Metric, F.Cu at (122.1, 77.0)
- added D20: LED, LED_SMD:LED_0402_1005Metric, F.Cu at (101.5, 109.7)
- added D21: LED, LED_SMD:LED_0402_1005Metric, F.Cu at (101.5, 111.7)
- added D22: LED, LED_SMD:LED_0402_1005Metric, F.Cu at (104.7, 95.8)
- added D23: LED, LED_SMD:LED_0402_1005Metric, F.Cu at (104.7, 97.8)
- added D24: LED, LED_SMD:LED_0402_1005Metric, F.Cu at (104.7, 99.8)
- added D25: LED, LED_SMD:LED_0402_1005Metric, F.Cu at (104.7, 101.8)
- added D26: LED, LED_SMD:LED_0402_1005Metric, F.Cu at (104.7, 103.8)
- added D27: LED, LED_SMD:LED_0402_1005Metric, F.Cu at (104.7, 105.7)
- added D28: LED, LED_SMD:LED_0402_1005Metric, F.Cu at (104.7, 107.7)
- added D29: LED, LED_SMD:LED_0402_1005Metric, F.Cu at (104.7, 109.7)
- added D30: LED, LED_SMD:LED_0402_1005Metric, F.Cu at (104.7, 111.7)
- added D31: LED, LED_SMD:LED_0402_1005Metric, F.Cu at (107.8, 95.8)
- added D32: LED, LED_SMD:LED_0402_1005Metric, F.Cu at (107.8, 97.8)
- added D33: LED, LED_SMD:LED_0402_1005Metric, F.Cu at (107.8, 99.8)
- added D34: LED, LED_SMD:LED_0402_1005Metric, F.Cu at (107.8, 101.8)
- added D35: LED, LED_SMD:LED_0402_1005Metric, F.Cu at (107.8, 103.8)
- added D4: LED, LED_SMD:LED_0402_1005Metric, F.Cu at (103.3, 77.0)
- added D5: LED, LED_SMD:LED_0402_1005Metric, F.Cu at (104.6, 77.0)
- added D6: LED, LED_SMD:LED_0402_1005Metric, F.Cu at (105.8, 77.0)
- added D7: LED, LED_SMD:LED_0402_1005Metric, F.Cu at (107.1, 77.0)
- added D8: LED, LED_SMD:LED_0402_1005Metric, F.Cu at (108.3, 77.0)
- added D9: LED, LED_SMD:LED_0402_1005Metric, F.Cu at (109.6, 77.0)
- added R15: 10k, Resistor_SMD:R_0402_1005Metric, F.Cu at (110.7, 95.8)
- added R16: 150, Resistor_SMD:R_0402_1005Metric, F.Cu at (110.7, 97.8)
- added R17: 150, Resistor_SMD:R_0402_1005Metric, F.Cu at (110.7, 99.8)
- added R18: 150, Resistor_SMD:R_0402_1005Metric, F.Cu at (110.7, 101.8)
- added R19: 150, Resistor_SMD:R_0402_1005Metric, F.Cu at (110.7, 103.8)
- added R20: 150, Resistor_SMD:R_0402_1005Metric, F.Cu at (110.7, 105.7)
- added R21: 150, Resistor_SMD:R_0402_1005Metric, F.Cu at (110.7, 107.7)
- added R22: 150, Resistor_SMD:R_0402_1005Metric, F.Cu at (110.7, 109.7)
- added R23: 150, Resistor_SMD:R_0402_1005Metric, F.Cu at (113.7, 95.8)
- added R24: 150, Resistor_SMD:R_0402_1005Metric, F.Cu at (113.7, 97.8)
- added R25: 150, Resistor_SMD:R_0402_1005Metric, F.Cu at (113.7, 99.8)
- added R26: 150, Resistor_SMD:R_0402_1005Metric, F.Cu at (113.7, 101.8)
- added R27: 150, Resistor_SMD:R_0402_1005Metric, F.Cu at (113.7, 103.8)
- added R28: 150, Resistor_SMD:R_0402_1005Metric, F.Cu at (113.7, 105.7)
- added R29: 150, Resistor_SMD:R_0402_1005Metric, F.Cu at (113.7, 107.7)
- added R30: 150, Resistor_SMD:R_0402_1005Metric, F.Cu at (113.7, 109.7)
- added R31: 150, Resistor_SMD:R_0402_1005Metric, F.Cu at (116.6, 95.8)
- added R32: 150, Resistor_SMD:R_0402_1005Metric, F.Cu at (116.6, 97.8)
- added R33: 150, Resistor_SMD:R_0402_1005Metric, F.Cu at (116.6, 99.8)
- added R34: 150, Resistor_SMD:R_0402_1005Metric, F.Cu at (116.6, 101.8)
- added R35: 150, Resistor_SMD:R_0402_1005Metric, F.Cu at (116.6, 103.8)
- added R36: 150, Resistor_SMD:R_0402_1005Metric, F.Cu at (116.6, 105.7)
- added R37: 150, Resistor_SMD:R_0402_1005Metric, F.Cu at (116.6, 107.7)
- added R38: 150, Resistor_SMD:R_0402_1005Metric, F.Cu at (116.6, 109.7)
- added R39: 150, Resistor_SMD:R_0402_1005Metric, F.Cu at (119.5, 95.8)
- added R40: 150, Resistor_SMD:R_0402_1005Metric, F.Cu at (119.5, 97.8)
- added R41: 150, Resistor_SMD:R_0402_1005Metric, F.Cu at (119.5, 99.8)
- added R42: 150, Resistor_SMD:R_0402_1005Metric, F.Cu at (119.5, 101.8)
- added R43: 150, Resistor_SMD:R_0402_1005Metric, F.Cu at (119.5, 103.8)
- added R44: 150, Resistor_SMD:R_0402_1005Metric, F.Cu at (119.5, 105.7)
- added R45: 150, Resistor_SMD:R_0402_1005Metric, F.Cu at (119.5, 107.7)
- added R46: 150, Resistor_SMD:R_0402_1005Metric, F.Cu at (119.5, 109.7)
- C25, C27: value 4.7uF -> 100nF; footprint Capacitor_SMD:C_0603_1608Metric -> Capacitor_SMD:C_0402_1005Metric
- C26, C28: value 100nF -> 4.7uF; footprint Capacitor_SMD:C_0402_1005Metric -> Capacitor_SMD:C_0603_1608Metric
- IC1: value FPGA_ICE40UP5K-SG48I -> FT2232HQ; footprint NB3_hindbrain:FPGA_ICE40UP5K-SG48I -> NB3_hindbrain:USBtoSerial_FT2232HQ
- IC2: value NOR_Flash_W25Q32JVSSIQ -> FPGA_ICE40UP5K-SG48I; footprint NB3_hindbrain:NOR_Flash_W25Q32JVSSIQ -> NB3_hindbrain:FPGA_ICE40UP5K-SG48I
- IC3: value FT232HL -> NOR_Flash_W25Q32JVSSIQ; footprint NB3_hindbrain:USBtoSPI_FT232HL -> NB3_hindbrain:NOR_Flash_W25Q32JVSSIQ; moved to B.Cu
- R14: value 10k -> 150
- moved IC1 29.0 mm to (97.1, 80.0)
- moved IC3 20.5 mm to (117.1, 80.0), turned to 180 degrees
- moved IC2 13.5 mm to (127.1, 80.0)
- moved R11 13.2 mm to (96.1, 74.0), turned to 0 degrees
- moved Y1 11.2 mm to (116.7, 84.7)
- moved R12 10.6 mm to (98.1, 74.0), turned to 0 degrees
- moved VR2 9.50 mm to (106.1, 80.0)
- moved C23 8.53 mm to (127.1, 74.5), turned to 180 degrees
- moved R14 7.81 mm to (125.1, 74.5), turned to 0 degrees
- moved C7 6.02 mm to (103.1, 83.5)
- moved R1 6.02 mm to (102.6, 86.0)
- moved R4 6.02 mm to (102.6, 85.0)
- moved U1 5.95 mm to (105.9, 84.9)
- moved C20 5.39 mm to (102.6, 74.5)
- moved C19 4.81 mm to (119.6, 84.5)
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Connections:
- C24 pad 1: Net-(IC1-VPP_2V5) -> GND
- C24 pad 2: GND -> +3V3
- C25 pad 1: +3V3 -> Net-(IC2-VPP_2V5)
- C26 pad 1: Net-(IC1-VCCPLL) -> +3V3
- C27 pad 1: Net-(IC1-VCCPLL) -> Net-(IC2-VCCPLL)
- C28 pad 1: GND -> Net-(IC2-VCCPLL)
- C28 pad 2: +3V3 -> GND
- D3 pad C: Net-(IC1-VPP_2V5) -> Net-(IC2-VPP_2V5)
- IC1 pad 1: +3V3 -> unconnected-(IC1-GND_1-Pad1)
- IC1 pad 10: /IOB_18A -> unconnected-(IC1-AGND-Pad10)
- IC1 pad 11: /IOB_20A -> unconnected-(IC1-GND_3-Pad11)
- IC1 pad 12: /IOB_22A -> unconnected-(IC1-VCORE_1-Pad12)
- IC1 pad 13: /IOB_24A -> unconnected-(IC1-TEST-Pad13)
- IC1 pad 14: /FLASH_SI -> unconnected-(IC1-RESET#-Pad14)
- IC1 pad 15: /FLASH_SCK -> unconnected-(IC1-GND_4-Pad15)
- IC1 pad 16: /FLASH_SSn -> unconnected-(IC1-ADBUS0-Pad16)
- IC1 pad 17: /FLASH_SO -> unconnected-(IC1-ADBUS1-Pad17)
- IC1 pad 18: /IOB_31B -> unconnected-(IC1-ADBUS2-Pad18)
- IC1 pad 19: /IOB_29B -> unconnected-(IC1-ADBUS3-Pad19)
- IC1 pad 2: /IOB_6A -> unconnected-(IC1-OSCI-Pad2)
- IC1 pad 20: /IOB_25B_G3 -> unconnected-(IC1-VCCIO_1-Pad20)
- IC1 pad 21: /IOB_23B -> unconnected-(IC1-ADBUS4-Pad21)
- IC1 pad 22: +3V3 -> unconnected-(IC1-ADBUS5-Pad22)
- IC1 pad 23: /IOT_37A -> unconnected-(IC1-ADBUS6-Pad23)
- IC1 pad 24: Net-(IC1-VPP_2V5) -> unconnected-(IC1-ADBUS7-Pad24)
- IC1 pad 25: /IOT_36B -> unconnected-(IC1-GND_5-Pad25)
- IC1 pad 26: /IOT_39A -> unconnected-(IC1-ACBUS0-Pad26)
- IC1 pad 27: /IOT_38B -> unconnected-(IC1-ACBUS1-Pad27)
- IC1 pad 28: /IOT_41A -> unconnected-(IC1-ACBUS2-Pad28)
- IC1 pad 29: Net-(IC1-VCCPLL) -> unconnected-(IC1-ACBUS3-Pad29)
- IC1 pad 3: /IOB_9B -> unconnected-(IC1-OSCO-Pad3)
- IC1 pad 30: +1V2 -> unconnected-(IC1-ACBUS4-Pad30)
- IC1 pad 31: /IOT_42B -> unconnected-(IC1-VCCIO_2-Pad31)
- IC1 pad 32: /IOT_43A -> unconnected-(IC1-ACBUS5-Pad32)
- IC1 pad 33: +3V3 -> unconnected-(IC1-ACBUS6-Pad33)
- IC1 pad 34: /IOT_44B -> unconnected-(IC1-ACBUS7-Pad34)
- IC1 pad 35: /IOT_46B_G0 -> unconnected-(IC1-GND_6-Pad35)
- IC1 pad 36: /IOT_48B -> unconnected-(IC1-SUSPEND#-Pad36)
- IC1 pad 37: /IOT_45A_G1 -> unconnected-(IC1-VCORE_2-Pad37)
- IC1 pad 38: /IOT_50B -> unconnected-(IC1-BDBUS0-Pad38)
- IC1 pad 39: /RGB0 -> unconnected-(IC1-BDBUS1-Pad39)
- IC1 pad 4: /IOB_8A -> unconnected-(IC1-VPHY-Pad4)
- IC1 pad 40: /RGB1 -> unconnected-(IC1-BDBUS2-Pad40)
- IC1 pad 41: /RGB2 -> unconnected-(IC1-BDBUS3-Pad41)
- IC1 pad 42: /IOT_51A -> unconnected-(IC1-VCCIO_3-Pad42)
- IC1 pad 43: /IOT_49A -> unconnected-(IC1-BDBUS4-Pad43)
- IC1 pad 44: /IOB_3B_G6 -> unconnected-(IC1-BDBUS5-Pad44)
- IC1 pad 45: /IOB_5B -> unconnected-(IC1-BDBUS6-Pad45)
- IC1 pad 46: /IOB_0A -> unconnected-(IC1-BDBUS7-Pad46)
- IC1 pad 47: /IOB_2A -> unconnected-(IC1-GND_7-Pad47)
- IC1 pad 48: /IOB_4A -> unconnected-(IC1-BCBUS0-Pad48)
- IC1 pad 49: GND -> unconnected-(IC1-VREGOUT-Pad49)
- IC1 pad 5: +1V2 -> unconnected-(IC1-GND_2-Pad5)
- IC1 pad 6: /IOB_13B -> unconnected-(IC1-REF-Pad6)
- IC1 pad 7: /CDONE -> unconnected-(IC1-DM-Pad7)
- IC1 pad 8: /CRESET_B -> unconnected-(IC1-DP-Pad8)
- IC1 pad 9: /IOB_16A -> unconnected-(IC1-VPLL-Pad9)
- IC2 pad 1: /FLASH_SSn -> +3V3
- IC2 pad 2: /FLASH_SO -> /IOB_6A
- IC2 pad 3: /FLASH_WPn -> /IOB_9B
- IC2 pad 4: GND -> /IOB_8A
- IC2 pad 5: /FLASH_SI -> +1V2
- IC2 pad 6: /FLASH_SCK -> /IOB_13B
- IC2 pad 7: /FLASH_HOLDn -> /CDONE
- IC2 pad 8: +3V3 -> /CRESET_B
- IC3 pad 1: unconnected-(IC3-XCSI-Pad1) -> /FLASH_SSn
- IC3 pad 2: unconnected-(IC3-XCSO-Pad2) -> /FLASH_SO
- IC3 pad 3: unconnected-(IC3-VPHY-Pad3) -> /FLASH_WPn
- IC3 pad 4: unconnected-(IC3-AGND_1-Pad4) -> GND
- IC3 pad 5: unconnected-(IC3-REF-Pad5) -> /FLASH_SI
- IC3 pad 6: unconnected-(IC3-DM-Pad6) -> /FLASH_SCK
- IC3 pad 7: unconnected-(IC3-DP-Pad7) -> /FLASH_HOLDn
- IC3 pad 8: unconnected-(IC3-VPLL-Pad8) -> +3V3
- J2 pad 1: GND -> +5V
- J2 pad 10: /IOB_13B -> /IOT_41A
- J2 pad 11: /IOB_16A -> /IOT_42B
- J2 pad 12: /IOB_18A -> /IOT_43A
- J2 pad 13: /IOB_20A -> /IOT_44B
- J2 pad 14: /IOB_22A -> /IOT_46B_G0
- J2 pad 15: /IOB_24A -> /IOT_48B
- J2 pad 16: /IOB_31B -> /IOT_45A_G1
- J2 pad 17: /IOB_29B -> /IOT_50B
- J2 pad 18: /IOB_25B_G3 -> /IOT_51A
- J2 pad 19: /IOB_23B -> /IOT_49A
- J2 pad 2: /IOB_3B_G6 -> /USB_5V
- J2 pad 20: GND -> +3V3
- J2 pad 3: /IOB_5B -> /RGB2
- J2 pad 4: /IOB_0A -> /RGB1
- J2 pad 5: /IOB_2A -> /RGB0
- J2 pad 6: /IOB_4A -> /IOT_37A
- J2 pad 7: /IOB_6A -> /IOT_36B
- J2 pad 8: /IOB_9B -> /IOT_39A
- J2 pad 9: /IOB_8A -> /IOT_38B
- J3 pad 1: +5V -> GND
- J3 pad 10: /IOT_41A -> /IOB_13B
- J3 pad 11: /IOT_42B -> /IOB_16A
- J3 pad 12: /IOT_43A -> /IOB_18A
- J3 pad 13: /IOT_44B -> /IOB_20A
- J3 pad 14: /IOT_46B_G0 -> /IOB_22A
- J3 pad 15: /IOT_48B -> /IOB_24A
- J3 pad 16: /IOT_45A_G1 -> /IOB_31B
- J3 pad 17: /IOT_50B -> /IOB_29B
- J3 pad 18: /IOT_51A -> /IOB_25B_G3
- J3 pad 19: /IOT_49A -> /IOB_23B
- J3 pad 2: /USB_5V -> /IOB_3B_G6
- J3 pad 20: +3V3 -> GND
- J3 pad 3: /RGB2 -> /IOB_5B
- J3 pad 4: /RGB1 -> /IOB_0A
- J3 pad 5: /RGB0 -> /IOB_2A
- J3 pad 6: /IOT_37A -> /IOB_4A
- J3 pad 7: /IOT_36B -> /IOB_6A
- J3 pad 8: /IOT_39A -> /IOB_9B
- J3 pad 9: /IOT_38B -> /IOB_8A
- R13 pad 2: Net-(IC1-VCCPLL) -> Net-(IC2-VCCPLL)
- R14 pad 1: /FLASH_HOLDn -> Net-(D4-K)
- R14 pad 2: +3V3 -> GND
