File: boxes/fpgas/NB3_hindbrain/NB3_hindbrain.kicad_pcb (KiCad board)
At the start: 4 copper layers, 57 x 22 mm, 122 parts, among them IC1 FT2232HQ, IC2 FPGA_ICE40UP5K-SG48I, IC3 NOR_Flash_W25Q32JVSSIQ, IC4 ADC_MCP3004-I-SL, J1 MicroUSB_10103594-0001LF, J2 Conn_01x20_Male, J3 Conn_01x20_Male, U1 EEPROM_93LC56BT-I-OT, Y1 Osc_12MHz_ECS-2520MV-120-BN-TR

Commit message: Work on NB£_hindbrain schematic
Parts:
- removed D10, D11, D12, D29, D30, D31, D32, D33, D34, D35, D5, D6, D7, D8, D9: LED, LED_SMD:LED_0402_1005Metric
- removed R14, R16, R17, R18, R19, R20, R21, R22, R39, R40, R41, R42, R43, R44, R45, R46: 150, Resistor_SMD:R_0402_1005Metric
- added C29: 4.7uF, Capacitor_SMD:C_0603_1608Metric, F.Cu at (119.6, 86.0)
- added C30: 100nF, Capacitor_SMD:C_0402_1005Metric, F.Cu at (119.6, 74.5)
- added LED1: CLMVC-FKA-CLBDGL7LBB79353, NB3_hindbrain:RGB_CLMVC-FKA-CLBDGL7LBB79353, F.Cu at (119.6, 80.0)
- added R47: 17k, Resistor_SMD:R_0402_1005Metric, F.Cu at (90.8, 95.1)
- added R48: 33k, Resistor_SMD:R_0402_1005Metric, F.Cu at (90.8, 97.1)
- added R49: 17k, Resistor_SMD:R_0402_1005Metric, F.Cu at (90.8, 99.1)
- added R50: 17k, Resistor_SMD:R_0402_1005Metric, F.Cu at (90.8, 101.0)
- added R51: 33k, Resistor_SMD:R_0402_1005Metric, F.Cu at (90.8, 103.0)
- added R52: 33k, Resistor_SMD:R_0402_1005Metric, F.Cu at (90.8, 105.0)
- added R53: 17k, Resistor_SMD:R_0402_1005Metric, F.Cu at (90.8, 107.0)
- added R54: 33k, Resistor_SMD:R_0402_1005Metric, F.Cu at (90.8, 109.0)
- C18: footprint Capacitor_SMD:C_0603_1608Metric -> Capacitor_SMD:C_0402_1005Metric
- C23: value 100nF -> 4.7uF; footprint Capacitor_SMD:C_0402_1005Metric -> Capacitor_SMD:C_0603_1608Metric
- C28: value 4.7uF -> 100nF; footprint Capacitor_SMD:C_0603_1608Metric -> Capacitor_SMD:C_0402_1005Metric
- D3: value Diode_1N4148WS-7-F -> LED; footprint NB3_hindbrain:Diode_1N4148WS-7-F -> LED_SMD:LED_0603_1608Metric
- D4: value LED -> Diode_1N4148WS-7-F; footprint LED_SMD:LED_0402_1005Metric -> NB3_hindbrain:Diode_1N4148WS-7-F
- J2, J3: value Conn_01x20_Male -> Conn_01x20_Pin
- R10: value 150 -> 10k
- R5: value 4.7k -> 12k (1%)
- R6: value 10k -> 1k
- R7: value 1k -> 150
- R8: value 150 -> 220
- R9: value 12k -> 220
- moved D20 37.3 mm to (115.1, 75.0), turned to 90 degrees
- moved D21 26.9 mm to (104.6, 85.0), turned to 90 degrees
- moved D28 25.0 mm to (115.1, 85.0), turned to 90 degrees
- moved D27 22.6 mm to (113.6, 85.0), turned to 90 degrees
- moved D26 20.2 mm to (112.1, 85.0), turned to 90 degrees
- moved D25 17.8 mm to (110.6, 85.0), turned to 90 degrees
- moved D24 15.4 mm to (109.1, 85.0), turned to 90 degrees
- moved D23 13.1 mm to (107.6, 85.0), turned to 90 degrees
- moved D4 11.4 mm to (97.0, 86.5), turned to 180 degrees
- moved D22 10.9 mm to (106.1, 85.0), turned to 90 degrees
- moved D13 10.2 mm to (104.6, 75.0)
- moved D14 9.96 mm to (106.1, 75.0)
- moved D15 9.71 mm to (107.6, 75.0)
- moved D16 9.47 mm to (109.1, 75.0)
- moved D17 9.22 mm to (110.6, 75.0)
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Connections:
- net /FLASH_HOLDn renamed /FLASH_HOLD
- net /FLASH_WPn renamed /FLASH_WP
- C18 pad 1: GND -> +1V8
- C18 pad 2: +1V8 -> GND
- C23 pad 1: GND -> +3V3
- C23 pad 2: +3V3 -> GND
- C25 pad 1: Net-(IC2-VPP_2V5) -> GND
- C25 pad 2: GND -> +3V3
- C26 pad 1: +3V3 -> Net-(IC2-VPP_2V5)
- C27 pad 1: Net-(IC2-VCCPLL) -> +3V3
- C7 pad 1: +3V3 -> GND
- C7 pad 2: GND -> +1V8
- C8 pad 1: GND -> +3V3
- C8 pad 2: +1V8 -> GND
- D13 pad 2: unconnected-(D13-A-Pad2) -> /IOB_22A
- D14 pad 2: unconnected-(D14-A-Pad2) -> /IOB_20A
- D15 pad 2: unconnected-(D15-A-Pad2) -> /IOB_18A
- D16 pad 2: unconnected-(D16-A-Pad2) -> /IOB_16A
- D17 pad 2: unconnected-(D17-A-Pad2) -> /IOB_13B
- D18 pad 2: unconnected-(D18-A-Pad2) -> /IOB_8A
- D19 pad 2: unconnected-(D19-A-Pad2) -> /IOB_9B
- D2 pad 2: +5V -> +3V3
- D20 pad 2: unconnected-(D20-A-Pad2) -> /IOB_6A
- D21 pad 2: unconnected-(D21-A-Pad2) -> /IOT_48B
- D22 pad 2: unconnected-(D22-A-Pad2) -> /IOT_44B
- D23 pad 2: unconnected-(D23-A-Pad2) -> /IOT_43A
- D24 pad 2: unconnected-(D24-A-Pad2) -> /IOT_42B
- D25 pad 2: unconnected-(D25-A-Pad2) -> /IOT_41A
- D26 pad 2: unconnected-(D26-A-Pad2) -> /IOT_38B
- D27 pad 2: unconnected-(D27-A-Pad2) -> /IOT_39A
- D28 pad 2: unconnected-(D28-A-Pad2) -> /IOT_36B
- FB1 pad 1: /FT_VPLL -> /FT_VPHY
- FB1 pad 2: Net-(FB1-Pad2) -> +3V3
- FB2 pad 1: /FT_VPHY -> /FT_VPLL
- FB2 pad 2: Net-(FB1-Pad2) -> +3V3
- IC1 pad 1: unconnected-(IC1-GND_1-Pad1) -> GND
- IC1 pad 10: unconnected-(IC1-AGND-Pad10) -> GND
- IC1 pad 11: unconnected-(IC1-GND_3-Pad11) -> GND
- IC1 pad 12: unconnected-(IC1-VCORE_1-Pad12) -> +1V8
- IC1 pad 13: unconnected-(IC1-TEST-Pad13) -> GND
- IC1 pad 14: unconnected-(IC1-RESET#-Pad14) -> Net-(IC1-RESET#)
- IC1 pad 15: unconnected-(IC1-GND_4-Pad15) -> GND
- IC1 pad 16: unconnected-(IC1-ADBUS0-Pad16) -> /FPGA_SCLK
- IC1 pad 17: unconnected-(IC1-ADBUS1-Pad17) -> /FLASH_MOSI
- IC1 pad 18: unconnected-(IC1-ADBUS2-Pad18) -> /FLASH_MISO
- IC1 pad 2: unconnected-(IC1-OSCI-Pad2) -> /CLK_12MHz
- IC1 pad 20: unconnected-(IC1-VCCIO_1-Pad20) -> +3V3
- IC1 pad 21: unconnected-(IC1-ADBUS4-Pad21) -> /FPGA_CS
- IC1 pad 23: unconnected-(IC1-ADBUS6-Pad23) -> /CDONE
- IC1 pad 24: unconnected-(IC1-ADBUS7-Pad24) -> /CRESET
- IC1 pad 25: unconnected-(IC1-GND_5-Pad25) -> GND
- IC1 pad 31: unconnected-(IC1-VCCIO_2-Pad31) -> +3V3
- IC1 pad 35: unconnected-(IC1-GND_6-Pad35) -> GND
- IC1 pad 37: unconnected-(IC1-VCORE_2-Pad37) -> +1V8
- IC1 pad 38: unconnected-(IC1-BDBUS0-Pad38) -> /UART_Tx
- IC1 pad 39: unconnected-(IC1-BDBUS1-Pad39) -> /UART_Rx
- IC1 pad 4: unconnected-(IC1-VPHY-Pad4) -> /FT_VPHY
- IC1 pad 42: unconnected-(IC1-VCCIO_3-Pad42) -> +3V3
- IC1 pad 47: unconnected-(IC1-GND_7-Pad47) -> GND
- IC1 pad 49: unconnected-(IC1-VREGOUT-Pad49) -> +1V8
- IC1 pad 5: unconnected-(IC1-GND_2-Pad5) -> GND
- IC1 pad 50: unconnected-(IC1-VREGIN-Pad50) -> +3V3
- IC1 pad 51: unconnected-(IC1-GND_8-Pad51) -> GND
- IC1 pad 54: unconnected-(IC1-BCBUS3-Pad54) -> /Rx_LED
- IC1 pad 55: unconnected-(IC1-BCBUS4-Pad55) -> /Tx_LED
- IC1 pad 56: unconnected-(IC1-VCCIO_4-Pad56) -> +3V3
- IC1 pad 59: unconnected-(IC1-BCBUS7-Pad59) -> +3V3
- IC1 pad 6: unconnected-(IC1-REF-Pad6) -> Net-(IC1-REF)
- IC1 pad 61: unconnected-(IC1-EEDATA-Pad61) -> /EEDATA
- IC1 pad 62: unconnected-(IC1-EECLK-Pad62) -> /EECLK
- IC1 pad 63: unconnected-(IC1-EECS-Pad63) -> /EECS
- IC1 pad 64: unconnected-(IC1-VCORE_3-Pad64) -> +1V8
- IC1 pad 7: unconnected-(IC1-DM-Pad7) -> /USB_DN
- IC1 pad 8: unconnected-(IC1-DP-Pad8) -> /USB_DP
- IC1 pad 9: unconnected-(IC1-VPLL-Pad9) -> /FT_VPLL
- IC2 pad 13: /IOB_24A -> unconnected-(IC2-IOB_24A-Pad13)
- IC2 pad 14: /FLASH_SI -> /FLASH_MOSI
- IC2 pad 15: /FLASH_SCK -> /FPGA_SCLK
- IC2 pad 16: /FLASH_SSn -> /FPGA_CS
- IC2 pad 17: /FLASH_SO -> /FLASH_MISO
- IC2 pad 18: /IOB_31B -> unconnected-(IC2-IOB_31B-Pad18)
- IC2 pad 19: /IOB_29B -> unconnected-(IC2-IOB_29B-Pad19)
- IC2 pad 20: /IOB_25B_G3 -> unconnected-(IC2-IOB_25B_G3-Pad20)
- IC2 pad 21: /IOB_23B -> unconnected-(IC2-IOB_23B-Pad21)
- IC2 pad 23: /IOT_37A -> unconnected-(IC2-IOT_37A-Pad23)
- IC2 pad 35: /IOT_46B_G0 -> unconnected-(IC2-IOT_46B_G0-Pad35)
- IC2 pad 37: /IOT_45A_G1 -> unconnected-(IC2-IOT_45A_G1-Pad37)
- IC2 pad 38: /IOT_50B -> unconnected-(IC2-IOT_50B-Pad38)
- IC2 pad 42: /IOT_51A -> unconnected-(IC2-IOT_51A-Pad42)
- IC2 pad 43: /IOT_49A -> unconnected-(IC2-IOT_49A-Pad43)
- IC2 pad 44: /IOB_3B_G6 -> unconnected-(IC2-IOB_3B_G6-Pad44)
- IC2 pad 8: /CRESET_B -> /CRESET
- IC3 pad 1: /FLASH_SSn -> /FPGA_CS
- IC3 pad 2: /FLASH_SO -> /FLASH_MISO
- IC3 pad 5: /FLASH_SI -> /FLASH_MOSI
- IC3 pad 6: /FLASH_SCK -> /FPGA_SCLK
- IC4 pad 1: unconnected-(IC4-CH0-Pad1) -> Net-(IC4-CH0)
- IC4 pad 10: unconnected-(IC4-DOUT-Pad10) -> /IOB_2A
- IC4 pad 11: unconnected-(IC4-CLK-Pad11) -> /IOB_4A
- IC4 pad 12: unconnected-(IC4-AGND-Pad12) -> GND
- IC4 pad 13: unconnected-(IC4-VREF-Pad13) -> +3V3
- IC4 pad 14: unconnected-(IC4-VDD-Pad14) -> +3V3
- IC4 pad 2: unconnected-(IC4-CH1-Pad2) -> Net-(IC4-CH1)
- IC4 pad 3: unconnected-(IC4-CH2-Pad3) -> Net-(IC4-CH2)
- IC4 pad 4: unconnected-(IC4-CH3-Pad4) -> Net-(IC4-CH3)
- IC4 pad 7: unconnected-(IC4-DGND-Pad7) -> GND
- IC4 pad 8: unconnected-(IC4-~{CS}/SHDN-Pad8) -> /IOB_5B
- IC4 pad 9: unconnected-(IC4-DIN-Pad9) -> /IOB_0A
- J2 pad 10: /IOT_41A -> /IOB_16A
- J2 pad 11: /IOT_42B -> /IOB_13B
- J2 pad 12: /IOT_43A -> /IOB_8A
- J2 pad 13: /IOT_44B -> /IOB_9B
- J2 pad 14: /IOT_46B_G0 -> /IOB_6A
- J2 pad 15: /IOT_48B -> /CRESET
- J2 pad 16: /IOT_45A_G1 -> /CDONE
- J2 pad 17: /IOT_50B -> GND
- J2 pad 18: /IOT_51A -> /CLK_12MHz
- J2 pad 19: /IOT_49A -> GND
- J2 pad 2: /USB_5V -> /UART_Tx
- J2 pad 3: /RGB2 -> GND
- J2 pad 4: /RGB1 -> /Analog_1
- J2 pad 5: /RGB0 -> /Analog_3
- J2 pad 6: /IOT_37A -> GND
- J2 pad 7: /IOT_36B -> /IOB_22A
- J2 pad 8: /IOT_39A -> /IOB_20A
- J2 pad 9: /IOT_38B -> /IOB_18A
- J3 pad 1: GND -> +5V
- J3 pad 10: /IOB_13B -> /IOT_41A
- J3 pad 11: /IOB_16A -> /IOT_42B
- J3 pad 12: /IOB_18A -> /IOT_43A
- J3 pad 13: /IOB_20A -> /IOT_44B
- J3 pad 14: /IOB_22A -> /IOT_48B
- J3 pad 15: /IOB_24A -> /FLASH_MOSI
- J3 pad 16: /IOB_31B -> /FPGA_SCLK
- J3 pad 17: /IOB_29B -> /FPGA_CS
- J3 pad 18: /IOB_25B_G3 -> /FLASH_MISO
- J3 pad 19: /IOB_23B -> GND
- J3 pad 2: /IOB_3B_G6 -> /UART_Rx
- J3 pad 20: GND -> +3V3
- J3 pad 3: /IOB_5B -> GND
- J3 pad 4: /IOB_0A -> /Analog_0
- J3 pad 5: /IOB_2A -> /Analog_2
- J3 pad 6: /IOB_4A -> GND
- J3 pad 7: /IOB_6A -> /IOT_36B
- J3 pad 8: /IOB_9B -> /IOT_39A
- J3 pad 9: /IOB_8A -> /IOT_38B
- R1 pad 2: /EECLK -> Net-(U1-DO)
- R10 pad 1: Net-(D2-K) -> +3V3
- R10 pad 2: GND -> /CRESET
- R12 pad 2: /FLASH_SSn -> /FPGA_CS
- R2 pad 2: /EEDATA_O -> /EECS
- R23 pad 1: Net-(D12-K) -> Net-(D13-K)
- R24 pad 1: Net-(D13-K) -> Net-(D14-K)
- R25 pad 1: Net-(D14-K) -> Net-(D15-K)
- R26 pad 1: Net-(D15-K) -> Net-(D16-K)
- R27 pad 1: Net-(D16-K) -> Net-(D17-K)
- R28 pad 1: Net-(D17-K) -> Net-(D18-K)
- R29 pad 1: Net-(D18-K) -> Net-(D19-K)
- R3 pad 1: /EEDATA_O -> /EEDATA
- R3 pad 2: /EEDATA_I -> Net-(U1-DO)
- R30 pad 1: Net-(D19-K) -> Net-(D20-K)
- R31 pad 1: Net-(D20-K) -> Net-(D21-K)
- R32 pad 1: Net-(D21-K) -> Net-(D22-K)
- R33 pad 1: Net-(D22-K) -> Net-(D23-K)
- R34 pad 1: Net-(D23-K) -> Net-(D24-K)
- R35 pad 1: Net-(D24-K) -> Net-(D25-K)
- R36 pad 1: Net-(D25-K) -> Net-(D26-K)
- R37 pad 1: Net-(D26-K) -> Net-(D27-K)
- R38 pad 1: Net-(D27-K) -> Net-(D28-K)
- R4 pad 2: /EECS -> /EECLK
- R5 pad 1: /USB_5V -> GND
- R5 pad 2: Net-(R5-Pad2) -> Net-(IC1-REF)
- R6 pad 1: Net-(R5-Pad2) -> +3V3
- R6 pad 2: GND -> Net-(IC1-RESET#)
- R7 pad 1: Net-(R5-Pad2) -> Net-(D1-K)
- R7 pad 2: unconnected-(R7-Pad2) -> GND
- R8 pad 1: Net-(D1-K) -> Net-(D2-K)
- R8 pad 2: GND -> /Rx_LED
- R9 pad 1: unconnected-(R9-Pad1) -> Net-(D3-K)
- R9 pad 2: GND -> /Tx_LED
- U1 pad 1: /EEDATA_O -> Net-(U1-DO)
- U1 pad 3: /EEDATA_I -> /EEDATA

Commit message: Finished NB3 Hindbrain schematic
Parts:
- removed D22, D23, D24, D25, D26, D27, D28: LED, LED_SMD:LED_0402_1005Metric
- added C31: 100nF, Capacitor_SMD:C_0402_1005Metric, F.Cu at (134.1, 79.5)
- added C32: 10uF, Capacitor_SMD:C_0402_1005Metric, F.Cu at (134.1, 78.5)
- added C33: 100nF, Capacitor_SMD:C_0402_1005Metric, F.Cu at (134.1, 77.5)
- added C34: 100nF, Capacitor_SMD:C_0402_1005Metric, F.Cu at (134.1, 76.5)
- added C35: 10uF, Capacitor_SMD:C_0402_1005Metric, F.Cu at (134.1, 83.5)
- added D10: LED, LED_SMD:LED_0402_1005Metric, F.Cu at (108.6, 77.0)
- added D11: LED, LED_SMD:LED_0402_1005Metric, F.Cu at (108.6, 83.0)
- added D12: LED, LED_SMD:LED_0402_1005Metric, F.Cu at (110.6, 77.0)
- added D5: Diode_1N4148WS-7-F, NB3_hindbrain:Diode_1N4148WS-7-F, F.Cu at (131.6, 77.5)
- added D6: LED, LED_SMD:LED_0402_1005Metric, F.Cu at (104.6, 77.0)
- added D7: LED, LED_SMD:LED_0402_1005Metric, F.Cu at (104.6, 83.0)
- added D8: LED, LED_SMD:LED_0402_1005Metric, F.Cu at (106.6, 77.0)
- added D9: LED, LED_SMD:LED_0402_1005Metric, F.Cu at (106.6, 83.0)
- added F1: MF-FSMF035X-2, NB3_hindbrain:PTC_MF-FSMF035X-2, F.Cu at (88.1, 77.5)
- added G1: LOGO, NB3_hindbrain:Logo_NBB_5mm, F.Cu at (107.1, 80.0)
- added G2: Logo_VK, NB3_hindbrain:Logo_VK_5mm, F.Cu at (116.1, 80.0)
- added IC5: MCP4812-E_SN, NB3_hindbrain:DAC_MCP4812-E-SN, B.Cu at (132.6, 80.0)
- added Q1: RUM001L02T2CL, NB3_hindbrain:MOSFET_Nch_SOT-723_RUM001L02T2CL, F.Cu at (104.6, 74.5)
- added Q10: RUM001L02T2CL, NB3_hindbrain:MOSFET_Nch_SOT-723_RUM001L02T2CL, F.Cu at (112.6, 85.5)
- added Q11: RUM001L02T2CL, NB3_hindbrain:MOSFET_Nch_SOT-723_RUM001L02T2CL, F.Cu at (114.6, 74.5)
- added Q12: RUM001L02T2CL, NB3_hindbrain:MOSFET_Nch_SOT-723_RUM001L02T2CL, F.Cu at (114.6, 85.5)
- added Q13: RUM001L02T2CL, NB3_hindbrain:MOSFET_Nch_SOT-723_RUM001L02T2CL, F.Cu at (116.6, 74.5)
- added Q14: RUM001L02T2CL, NB3_hindbrain:MOSFET_Nch_SOT-723_RUM001L02T2CL, F.Cu at (116.6, 85.5)
- added Q15: RUM001L02T2CL, NB3_hindbrain:MOSFET_Nch_SOT-723_RUM001L02T2CL, F.Cu at (118.6, 74.5)
- added Q16: RUM001L02T2CL, NB3_hindbrain:MOSFET_Nch_SOT-723_RUM001L02T2CL, F.Cu at (118.6, 85.5)
- added Q2: RUM001L02T2CL, NB3_hindbrain:MOSFET_Nch_SOT-723_RUM001L02T2CL, F.Cu at (104.6, 85.5)
- added Q3: RUM001L02T2CL, NB3_hindbrain:MOSFET_Nch_SOT-723_RUM001L02T2CL, F.Cu at (106.6, 74.5)
- added Q4: RUM001L02T2CL, NB3_hindbrain:MOSFET_Nch_SOT-723_RUM001L02T2CL, F.Cu at (106.6, 85.5)
- added Q5: RUM001L02T2CL, NB3_hindbrain:MOSFET_Nch_SOT-723_RUM001L02T2CL, F.Cu at (108.6, 74.5)
- added Q6: RUM001L02T2CL, NB3_hindbrain:MOSFET_Nch_SOT-723_RUM001L02T2CL, F.Cu at (108.6, 85.5)
- added Q7: RUM001L02T2CL, NB3_hindbrain:MOSFET_Nch_SOT-723_RUM001L02T2CL, F.Cu at (110.6, 74.5)
- added Q8: RUM001L02T2CL, NB3_hindbrain:MOSFET_Nch_SOT-723_RUM001L02T2CL, F.Cu at (110.6, 85.5)
- added Q9: RUM001L02T2CL, NB3_hindbrain:MOSFET_Nch_SOT-723_RUM001L02T2CL, F.Cu at (112.6, 74.5)
- added R14: 100, Resistor_SMD:R_0402_1005Metric, F.Cu at (134.1, 81.5)
- added R16: 3M3, Resistor_SMD:R_0402_1005Metric, F.Cu at (104.6, 73.0)
- added R17: 3M3, Resistor_SMD:R_0402_1005Metric, F.Cu at (104.6, 87.0)
- added R18: 680, Resistor_SMD:R_0402_1005Metric, F.Cu at (104.6, 76.0)
- added R19: 680, Resistor_SMD:R_0402_1005Metric, F.Cu at (104.6, 84.0)
- added R20: 3M3, Resistor_SMD:R_0402_1005Metric, F.Cu at (106.6, 73.0)
- added R21: 3M3, Resistor_SMD:R_0402_1005Metric, F.Cu at (106.6, 87.0)
- added R22: 17k, Resistor_SMD:R_0402_1005Metric, F.Cu at (134.1, 80.5)
- added R39: 680, Resistor_SMD:R_0402_1005Metric, F.Cu at (110.6, 84.0)
- added R40: 3M3, Resistor_SMD:R_0402_1005Metric, F.Cu at (112.6, 73.0)
- added R41: 3M3, Resistor_SMD:R_0402_1005Metric, F.Cu at (112.6, 87.0)
- added R42: 680, Resistor_SMD:R_0402_1005Metric, F.Cu at (112.6, 76.0)
- added R43: 680, Resistor_SMD:R_0402_1005Metric, F.Cu at (112.6, 84.0)
- added R44: 3M3, Resistor_SMD:R_0402_1005Metric, F.Cu at (114.6, 73.0)
- added R45: 3M3, Resistor_SMD:R_0402_1005Metric, F.Cu at (114.6, 87.0)
- added R46: 680, Resistor_SMD:R_0402_1005Metric, F.Cu at (114.6, 76.0)
- added R55: 680, Resistor_SMD:R_0402_1005Metric, F.Cu at (118.6, 84.0)
- C22: value 10uF -> 4.7uF
- C23: value 4.7uF -> 10uF
- C25: value 100nF -> 4.7uF; footprint Capacitor_SMD:C_0402_1005Metric -> Capacitor_SMD:C_0603_1608Metric
- C26: value 4.7uF -> 100nF; footprint Capacitor_SMD:C_0603_1608Metric -> Capacitor_SMD:C_0402_1005Metric
- C30: value 100nF -> 10uF; footprint Capacitor_SMD:C_0402_1005Metric -> Capacitor_SMD:C_0603_1608Metric
- D4: value Diode_1N4148WS-7-F -> PRTR5V0U2F,115; footprint NB3_hindbrain:Diode_1N4148WS-7-F -> NB3_hindbrain:ESD_Diodes_PRTR5V0U2F-115
- R10: value 10k -> 120:1%
- R13: value 100 -> 10k
- R23, R25, R27, R29: value 150 -> 33k
- R24, R26, R28: value 150 -> 17k
- R30, R31, R34, R35, R38: value 150 -> 680
- R32, R33, R36, R37: value 150 -> 3M3
- R47, R50: value 17k -> 680
- R48, R52: value 33k -> 3M3
- R49, R53: value 17k -> 3M3
- R51, R54: value 33k -> 680
- VR1: value LDO_3v3_LM1117IMPX-3.3 -> LD1117S12TR; footprint NB3_hindbrain:LDO_3v3_LM1117IMPX-3.3 -> NB3_hindbrain:LDO_1v2_LD1117S12TR
- VR2: value LDO_1v2_AP7217D-12YG-13 -> LDO_3v3_LM1117IMPX-3.3; footprint NB3_hindbrain:LDO_1v2_AP7217D-12YG-13 -> NB3_hindbrain:LDO_3v3_LM1117IMPX-3.3
- moved R9 43.7 mm to (131.6, 82.0)
- moved R54 43.1 mm to (118.6, 76.0)
- moved R52 42.4 mm to (118.6, 73.0), turned to 180 degrees
- moved R50 35.9 mm to (116.6, 76.0)
- moved R48 35.2 mm to (116.6, 73.0), turned to 180 degrees
- moved R30 34.5 mm to (106.6, 76.0), turned to 180 degrees
- moved R38 34.2 mm to (110.6, 76.0)
- moved R53 34.2 mm to (118.6, 87.0), turned to 180 degrees
- moved R36 33.3 mm to (110.6, 73.0), turned to 180 degrees
- moved R51 32.0 mm to (116.6, 84.0), turned to 180 degrees
- moved R49 28.4 mm to (116.6, 87.0), turned to 180 degrees
- moved R34 27.0 mm to (108.6, 76.0), turned to 180 degrees
- moved R29 26.2 mm to (129.1, 86.5)
- moved R47 26.2 mm to (114.6, 84.0), turned to 180 degrees
- moved R32 26.0 mm to (108.6, 73.0), turned to 180 degrees
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Connections:
- C14 pad 1: +5V -> +3V3
- C15 pad 1: +3V3 -> +5V
- C16 pad 1: +5V -> +3V3
- C17 pad 1: +3V3 -> +5V
- C19 pad 1: +1V2 -> +3V3
- C20 pad 1: +3V3 -> +1V2
- C21 pad 1: +1V2 -> +3V3
- C23 pad 1: +3V3 -> +1V2
- C25 pad 1: GND -> Net-(IC2-VPP_2V5)
- C25 pad 2: +3V3 -> GND
- C26 pad 1: Net-(IC2-VPP_2V5) -> +3V3
- C27 pad 1: +3V3 -> Net-(IC2-VCCPLL)
- C28 pad 1: Net-(IC2-VCCPLL) -> GND
- C28 pad 2: GND -> +3V3
- D13 pad 2: /IOB_22A -> +3V3
- D14 pad 2: /IOB_20A -> +3V3
- D15 pad 2: /IOB_18A -> +3V3
- D16 pad 2: /IOB_16A -> +3V3
- D17 pad 2: /IOB_13B -> +3V3
- D18 pad 2: /IOB_8A -> +3V3
- D19 pad 2: /IOB_9B -> +3V3
- D20 pad 2: /IOB_6A -> +3V3
- D21 pad 2: /IOT_48B -> +3V3
- IC2 pad 13: unconnected-(IC2-IOB_24A-Pad13) -> /IOB_24A
- IC2 pad 18: unconnected-(IC2-IOB_31B-Pad18) -> /IOB_31B
- IC2 pad 19: unconnected-(IC2-IOB_29B-Pad19) -> /IOB_29B
- IC2 pad 21: unconnected-(IC2-IOB_23B-Pad21) -> /IOB_23B
- IC2 pad 35: unconnected-(IC2-IOT_46B_G0-Pad35) -> /CLK_12MHz
- IC2 pad 44: unconnected-(IC2-IOB_3B_G6-Pad44) -> /IOB_3B_G6
- J1 pad 2: /USB_DN -> /USB_DN_preESD
- J1 pad 3: /USB_DP -> /USB_DP_preESD
- J2 pad 1: +5V -> /USB_5V
- J2 pad 15: /CRESET -> /IOB_3B_G6
- J2 pad 16: /CDONE -> GND
- J2 pad 17: GND -> /A_in_2
- J2 pad 18: /CLK_12MHz -> /A_in_0
- J2 pad 19: GND -> /A_out_0
- J2 pad 2: /UART_Tx -> GND
- J2 pad 3: GND -> /FLASH_MISO
- J2 pad 4: /Analog_1 -> /FPGA_CS
- J2 pad 5: /Analog_3 -> /FPGA_SCLK
- J2 pad 6: GND -> /FLASH_MOSI
- J3 pad 1: +5V -> /USB_5V
- J3 pad 15: /FLASH_MOSI -> /CLK_12MHz
- J3 pad 16: /FPGA_SCLK -> GND
- J3 pad 17: /FPGA_CS -> /A_in_3
- J3 pad 18: /FLASH_MISO -> /A_in_1
- J3 pad 19: GND -> /A_out_1
- J3 pad 2: /UART_Rx -> GND
- J3 pad 3: GND -> /UART_Tx
- J3 pad 4: /Analog_0 -> /UART_Rx
- J3 pad 5: /Analog_2 -> /CRESET
- J3 pad 6: GND -> /CDONE
- R10 pad 1: +3V3 -> +1V2
- R10 pad 2: /CRESET -> GND
- R11 pad 2: /FLASH_WP -> /CRESET
- R12 pad 2: /FPGA_CS -> /FLASH_WP
- R13 pad 1: +1V2 -> +3V3
- R13 pad 2: Net-(IC2-VCCPLL) -> /FPGA_CS
- R23 pad 1: Net-(D13-K) -> GND
- R23 pad 2: GND -> Net-(IC4-CH0)
- R24 pad 1: Net-(D14-K) -> Net-(IC4-CH1)
- R24 pad 2: GND -> /A_in_1
- R25 pad 1: Net-(D15-K) -> GND
- R25 pad 2: GND -> Net-(IC4-CH1)
- R26 pad 1: Net-(D16-K) -> Net-(IC4-CH2)
- R26 pad 2: GND -> /A_in_2
- R27 pad 1: Net-(D17-K) -> GND
- R27 pad 2: GND -> Net-(IC4-CH2)
- R28 pad 1: Net-(D18-K) -> Net-(IC4-CH3)
- R28 pad 2: GND -> /A_in_3
- R29 pad 1: Net-(D19-K) -> GND
- R29 pad 2: GND -> Net-(IC4-CH3)
- R30 pad 1: Net-(D20-K) -> Net-(D8-K)
- R30 pad 2: GND -> Net-(Q3-D)
- R31 pad 1: Net-(D21-K) -> Net-(D9-K)
- R31 pad 2: GND -> Net-(Q4-D)
- R32 pad 1: Net-(D22-K) -> /IOB_18A
- R33 pad 1: Net-(D23-K) -> /IOT_38B
- R34 pad 2: GND -> Net-(Q5-D)
- R35 pad 2: GND -> Net-(Q6-D)
- R36 pad 1: Net-(D26-K) -> /IOB_16A
- R37 pad 1: Net-(D27-K) -> /IOT_41A
- R38 pad 2: GND -> Net-(Q7-D)
- R47 pad 1: Net-(IC4-CH1) -> Net-(D17-K)
- R47 pad 2: /Analog_1 -> Net-(Q12-D)
- R48 pad 1: GND -> /IOB_9B
- R48 pad 2: Net-(IC4-CH1) -> GND
- R49 pad 1: Net-(IC4-CH2) -> /IOT_44B
- R49 pad 2: /Analog_2 -> GND
- R50 pad 1: Net-(IC4-CH0) -> Net-(D18-K)
- R50 pad 2: /Analog_0 -> Net-(Q13-D)
- R51 pad 1: GND -> Net-(D19-K)
- R51 pad 2: Net-(IC4-CH0) -> Net-(Q14-D)
- R52 pad 1: GND -> /IOB_6A
- R52 pad 2: Net-(IC4-CH2) -> GND
- R53 pad 1: Net-(IC4-CH3) -> /IOT_48B
- R53 pad 2: /Analog_3 -> GND
- R54 pad 1: GND -> Net-(D20-K)
- R54 pad 2: Net-(IC4-CH3) -> Net-(Q15-D)
- VR1 pad 2: +3V3 -> +1V2
- VR1 pad 3: +5V -> +3V3
- VR1 pad 4: +3V3 -> +1V2
- VR2 pad 3: +1V2 -> +5V
Routing:
- net /USB_DN: track 6.96 -> 0.00 mm
- net /USB_DP: track 6.90 -> 0.00 mm
- net /FT_VPHY: track 5.81 -> 0.00 mm
- net /IOT_36B: track 0.00 -> 5.57 mm
- net /IOB_22A: track 0.00 -> 5.55 mm
- net /IOT_39A: track 0.00 -> 5.01 mm
- net /IOB_20A: track 0.00 -> 5.01 mm
- net /IOT_38B: track 0.00 -> 4.47 mm
- net /IOB_18A: track 0.00 -> 4.47 mm
- net /IOT_41A: track 0.00 -> 3.93 mm
- net /IOB_16A: track 0.00 -> 3.93 mm
- net /IOT_42B: track 0.00 -> 3.39 mm
- net /IOB_13B: track 0.00 -> 3.39 mm
- net /IOB_8A: track 0.00 -> 2.82 mm
- net /IOT_43A: track 0.00 -> 2.82 mm
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Other:
- board text added: "NB3 Hindbrain"
- board text added: "rev 0.0.1"

Commit message: Work on NB3 Hindbrain routing...
Parts:
- removed R10: 120:1%, Resistor_SMD:R_0402_1005Metric
- C11, C18, C7, IC3, R2, R4, Y1: moved to F.Cu
- C23, R5: moved to B.Cu
- D2, D3: footprint LED_SMD:LED_0603_1608Metric -> LED_SMD:LED_0402_1005Metric
- R7: value 150 -> 330
- R8, R9: value 220 -> 680
- moved R9 35.9 mm to (96.6, 74.0)
- moved D3 33.1 mm to (95.3, 72.8)
- moved C21 29.4 mm to (97.5, 83.5)
- moved C19 26.5 mm to (98.8, 82.9), turned to -90 degrees
- moved R6 23.3 mm to (82.3, 64.8)
- moved C23 22.8 mm to (108.7, 78.4), turned to 90 degrees
- moved C15 21.2 mm to (89.3, 74.8), turned to 180 degrees
- moved C17 21.2 mm to (89.6, 76.1), turned to 180 degrees
- moved C22 20.7 mm to (110.8, 80.0), turned to -90 degrees
- moved C13 18.5 mm to (70.8, 77.3)
- moved D2 18.3 mm to (97.8, 72.8), turned to 180 degrees
- moved FB1 18.2 mm to (71.1, 79.3)
- moved R7 17.6 mm to (81.6, 69.8)
- moved U1 16.6 mm to (93.6, 74.6)
- moved R8 16.5 mm to (98.6, 74.0), turned to 180 degrees
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Connections:
- D1 pad 2: +5V -> /USB_5V
- IC2 pad 20: unconnected-(IC2-IOB_25B_G3-Pad20) -> /IOB_25B_G3
- J2 pad 3: /FLASH_MISO -> /CLK_12MHz
- J2 pad 4: /FPGA_CS -> /CRESET
- J2 pad 5: /FPGA_SCLK -> /UART_Tx
- J2 pad 6: /FLASH_MOSI -> /UART_Rx
- J3 pad 15: /CLK_12MHz -> /IOB_25B_G3
- J3 pad 3: /UART_Tx -> /FPGA_SCLK
- J3 pad 4: /UART_Rx -> /FLASH_MOSI
- J3 pad 5: /CRESET -> /FLASH_MISO
- J3 pad 6: /CDONE -> /FPGA_CS
Routing:
- net +3V3: track 0.00 -> 83.8 mm, vias 0 -> 20
- net GND: track 0.00 -> 38.8 mm, vias 0 -> 20
- net +1V8: track 0.00 -> 28.8 mm
- net /USB_5V: track 0.00 -> 27.1 mm, vias 0 -> 4
- net +5V: track 0.00 -> 9.60 mm, vias 0 -> 3
- net /CLK_12MHz: track 0.00 -> 8.72 mm
- net /EECS: track 0.00 -> 6.70 mm, vias 0 -> 1
- net /FPGA_SCLK: track 0.00 -> 6.57 mm
- net /FPGA_CS: track 0.00 -> 5.66 mm
- net /FLASH_MISO: track 0.00 -> 5.23 mm
- net /FLASH_MOSI: track 0.00 -> 4.49 mm
- net /USB_DP: track 0.00 -> 3.89 mm
- net /USB_DN: track 0.00 -> 3.74 mm
- net /EECLK: track 0.00 -> 3.55 mm, vias 0 -> 1
- net /EEDATA: track 0.00 -> 3.52 mm, vias 0 -> 1
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- added copper zone on In2.Cu, net +3V3
- added copper zone on B.Cu, net GND
- added copper zone on F.Cu, net GND
- added copper zone on In1.Cu, net GND
Other:
- board size 57 x 22 mm -> 57 x 22.5 mm
- board text added: "12"
- board text added: "3v3"
- board text added: "5V"
- board text added: "A0"
- board text added: "A1"
- board text added: "A2"
- board text added: "A3"
- board text added: "CK"
- board text added: "CS"
- board text added: "D0"
- board text added: "D1"
- board text added: "For Research and Education ONLY"
- board text added: "Gnd"
- board text added: "L0"
- board text added: "L1"
- board text added: "L2"
- board text added: "L3"
- board text added: "L4"
- board text added: "L5"
- board text added: "L6"
- board text added: "L7"
- board text added: "LG"
- board text added: "R0"
- board text added: "R1"
- board text added: "R2"
- board text added: "R3"
- board text added: "R4"
- board text added: "R5"
- board text added: "R6"
- board text added: "R7"
- board text added: "RG"
- board text added: "Rst"
- board text added: "Rx"
- board text added: "SI"
- board text added: "SO"
- board text added: "Tx"
- board text added: "locked"

Commit message: More work on NB£ Hindbrain wiring...FTDI done
Parts:
- C28: moved to F.Cu
- R6: moved to B.Cu
- moved R12 44.9 mm to (139.6, 87.6)
- moved G2 36.0 mm to (81.3, 88.5)
- moved Y1 27.4 mm to (115.8, 80.0), turned to 0 degrees
- moved C2 22.9 mm to (100.9, 75.9), turned to 180 degrees
- moved R6 22.1 mm to (90.9, 85.1)
- moved R11 19.5 mm to (96.2, 86.8), turned to 90 degrees
- moved C13 18.6 mm to (88.7, 82.7), turned to -90 degrees
- moved FB2 17.5 mm to (87.1, 82.7), turned to -90 degrees
- moved C8 17.3 mm to (89.8, 73.5)
- moved FB1 16.7 mm to (87.1, 74.5), turned to 90 degrees
- moved C9 15.3 mm to (89.9, 82.3), turned to -90 degrees
- moved C4 14.8 mm to (102.4, 84.2)
- moved C1 10.3 mm to (90.0, 74.8), turned to 90 degrees
- moved C28 7.74 mm to (100.3, 85.8), turned to 180 degrees
- moved C5 7.55 mm to (88.7, 74.5), turned to 90 degrees
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Connections:
- IC1 pad 65: unconnected-(IC1-TP-Pad65) -> GND
Routing:
- net +3V3: track 83.8 -> 133.4 mm, vias 20 -> 23
- net GND: track 38.8 -> 62.7 mm, vias 20 -> 29
- net /CRESET: track 0.00 -> 18.2 mm, vias 0 -> 1
- net /UART_Tx: track 0.00 -> 15.1 mm, vias 0 -> 1
- net /UART_Rx: track 0.00 -> 13.2 mm, vias 0 -> 1
- net /CLK_12MHz: track 8.72 -> 0.00 mm
- net /FT_VPHY: track 0.00 -> 6.84 mm
- net +1V2: track 0.00 -> 6.30 mm
- net /FT_VPLL: track 0.00 -> 6.05 mm
- net Net-(IC1-RESET#): track 0.00 -> 4.11 mm, vias 0 -> 1
- net +1V8: track 28.8 -> 32.8 mm, vias 0 -> 1
- net /EECS: track 6.70 -> 4.02 mm
- net /EECLK: track 3.55 -> 5.86 mm
- net /CDONE: track 0.00 -> 1.15 mm, vias 0 -> 1
- net /USB_5V: track 27.1 -> 27.7 mm
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
Commit message: More wiring...
Parts:
- C30, C6: moved to B.Cu
- moved C30 16.6 mm to (110.1, 83.0), turned to 180 degrees
- moved C6 15.2 mm to (110.8, 77.6), turned to -90 degrees
- moved C20 0.58 mm to (108.7, 80.4)
- moved C23 0.50 mm to (108.7, 77.9)
- moved G1 0.45 mm to (107.3, 80.0)
- moved G2 0.35 mm to (81.6, 88.3)
Routing:
- net +3V3: track 133.4 -> 149.5 mm, vias 23 -> 26
- net GND: track 62.7 -> 66.6 mm
- net +1V2: track 6.30 -> 9.53 mm

Commit message: Hmm....wiring chaos (NB3 Hindbrain)
Parts:
- removed C35: 10uF, Capacitor_SMD:C_0402_1005Metric
- added C36: 10uF, Capacitor_SMD:C_0603_1608Metric, B.Cu at (126.1, 73.8)
- added C37: 100nF, Capacitor_SMD:C_0402_1005Metric, F.Cu at (124.3, 85.5)
- added C38: 100nF, Capacitor_SMD:C_0402_1005Metric, F.Cu at (125.3, 74.5)
- added C39: 10uF, Capacitor_SMD:C_0603_1608Metric, B.Cu at (123.6, 85.3)
- C18: value 3.3uF -> 4.7uF; footprint Capacitor_SMD:C_0402_1005Metric -> Capacitor_SMD:C_0603_1608Metric
- C27, C29, C31, C33, C34, R14, R23, R25, R27, R29: moved to B.Cu
- C32: footprint Capacitor_SMD:C_0402_1005Metric -> Capacitor_SMD:C_0603_1608Metric
- D1: footprint LED_SMD:LED_0603_1608Metric -> LED_SMD:LED_0402_1005Metric
- moved C31 36.7 mm to (110.8, 77.6), turned to 90 degrees
- moved C34 34.1 mm to (112.6, 85.3), turned to -90 degrees
- moved D5 25.1 mm to (119.3, 80.0)
- moved R23 23.8 mm to (112.8, 74.2), turned to -90 degrees
- moved R22 23.5 mm to (127.8, 72.7)
- moved C26 23.2 mm to (117.7, 80.0), turned to 90 degrees
- moved C10 23.0 mm to (127.3, 74.5), turned to -90 degrees
- moved C27 21.5 mm to (125.8, 83.3)
- moved R25 21.3 mm to (114.6, 74.2), turned to -90 degrees
- moved R14 20.6 mm to (126.2, 84.8), turned to 90 degrees
- moved C25 16.8 mm to (121.2, 85.9), turned to -90 degrees
- moved R29 16.2 mm to (118.6, 74.2), turned to -90 degrees
- moved R27 16.0 mm to (116.6, 74.2), turned to -90 degrees
- moved R12 15.9 mm to (131.4, 74.0), turned to -90 degrees
- moved R26 14.4 mm to (125.2, 72.7)
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Connections:
- IC2 pad V49_1: (no net) -> GND
- IC2 pad V49_10: (no net) -> GND
- IC2 pad V49_11: (no net) -> GND
- IC2 pad V49_12: (no net) -> GND
- IC2 pad V49_13: (no net) -> GND
- IC2 pad V49_14: (no net) -> GND
- IC2 pad V49_15: (no net) -> GND
- IC2 pad V49_16: (no net) -> GND
- IC2 pad V49_17: (no net) -> GND
- IC2 pad V49_18: (no net) -> GND
- IC2 pad V49_19: (no net) -> GND
- IC2 pad V49_2: (no net) -> GND
- IC2 pad V49_20: (no net) -> GND
- IC2 pad V49_21: (no net) -> GND
- IC2 pad V49_3: (no net) -> GND
- IC2 pad V49_4: (no net) -> GND
- IC2 pad V49_5: (no net) -> GND
- IC2 pad V49_6: (no net) -> GND
- IC2 pad V49_7: (no net) -> GND
- IC2 pad V49_8: (no net) -> GND
- IC2 pad V49_9: (no net) -> GND
Routing:
- net /CLK_12MHz: track 0.00 -> 52.6 mm, vias 0 -> 5
- net +1V2: track 9.53 -> 59.2 mm, vias 0 -> 6
- net GND: track 66.6 -> 107.8 mm, vias 29 -> 31
- net +3V3: track 149.5 -> 186.5 mm, vias 26 -> 28
- net /IOT_36B: track 5.57 -> 31.3 mm, vias 0 -> 3
- net /IOT_39A: track 5.01 -> 28.9 mm, vias 0 -> 3
- net /IOT_42B: track 3.39 -> 26.8 mm, vias 0 -> 3
- net /IOB_22A: track 6.70 -> 28.8 mm, vias 0 -> 3
- net /IOT_38B: track 4.47 -> 26.5 mm, vias 0 -> 3
- net /IOT_43A: track 2.82 -> 24.6 mm, vias 0 -> 3
- net /IOB_20A: track 6.16 -> 26.4 mm, vias 0 -> 3
- net /IOT_41A: track 3.93 -> 24.0 mm, vias 0 -> 3
- net /IOT_44B: track 2.52 -> 22.6 mm, vias 0 -> 3
- net /IOB_18A: track 5.62 -> 23.9 mm, vias 0 -> 3
- net /IOB_16A: track 5.08 -> 21.5 mm, vias 0 -> 3
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Other:
- board text added: "Hz"
- board text added: "PWR"
- board text removed: "12"
- board text removed: "locked"
