File: boxes/fpgas/NB3_hindbrain/NB3_hindbrain.kicad_pcb (KiCad board)
At the start: 4 copper layers, 57 x 22.5 mm, 147 parts, among them IC1 FT2232HQ, IC2 FPGA_ICE40UP5K-SG48I, IC3 NOR_Flash_W25Q32JVSSIQ, IC4 ADC_MCP3004-I-SL, IC5 MCP4812-E_SN, J1 MicroUSB_10103594-0001LF, J2 Conn_01x20_Pin, J3 Conn_01x20_Pin, Q1 RUM001L02T2CL, Q10 RUM001L02T2CL, Q11 RUM001L02T2CL, Q12 RUM001L02T2CL, Q13 RUM001L02T2CL, Q14 RUM001L02T2CL, Q15 RUM001L02T2CL, Q16 RUM001L02T2CL, Q2 RUM001L02T2CL, Q3 RUM001L02T2CL, Q4 RUM001L02T2CL, Q5 RUM001L02T2CL, Q6 RUM001L02T2CL, Q7 RUM001L02T2CL, Q8 RUM001L02T2CL, Q9 RUM001L02T2CL, U1 EEPROM_93LC56BT-I-OT, Y1 Osc_12MHz_ECS-2520MV-120-BN-TR

Commit message: Wiring progress...
Parts:
- moved R22 1.02 mm to (128.8, 72.6), turned to 180 degrees
- moved R24 1.02 mm to (128.8, 87.4), turned to 180 degrees
- moved R28 1.02 mm to (126.2, 87.4), turned to 180 degrees
- moved R26 1.02 mm to (126.2, 72.7), turned to 180 degrees
Connections:
- IC1 pad 65: GND -> unconnected-(IC1-TP-Pad65)
- IC2 pad V49_1: GND -> (no net)
- IC2 pad V49_10: GND -> (no net)
- IC2 pad V49_11: GND -> (no net)
- IC2 pad V49_12: GND -> (no net)
- IC2 pad V49_13: GND -> (no net)
- IC2 pad V49_14: GND -> (no net)
- IC2 pad V49_15: GND -> (no net)
- IC2 pad V49_16: GND -> (no net)
- IC2 pad V49_17: GND -> (no net)
- IC2 pad V49_18: GND -> (no net)
- IC2 pad V49_19: GND -> (no net)
- IC2 pad V49_2: GND -> (no net)
- IC2 pad V49_20: GND -> (no net)
- IC2 pad V49_21: GND -> (no net)
- IC2 pad V49_3: GND -> (no net)
- IC2 pad V49_4: GND -> (no net)
- IC2 pad V49_5: GND -> (no net)
- IC2 pad V49_6: GND -> (no net)
- IC2 pad V49_7: GND -> (no net)
- IC2 pad V49_8: GND -> (no net)
- IC2 pad V49_9: GND -> (no net)
- IC4 pad 10: /IOB_2A -> /IOB_31B
- IC4 pad 11: /IOB_4A -> /IOB_24A
- IC4 pad 8: /IOB_5B -> /IOB_23B
- IC4 pad 9: /IOB_0A -> /IOB_29B
- IC5 pad 2: /IOB_24A -> /IOB_2A
- IC5 pad 3: /IOB_31B -> /IOB_0A
- IC5 pad 4: /IOB_29B -> /IOB_5B
- IC5 pad 5: /IOB_23B -> /IOB_4A
- J2 pad 10: /IOB_16A -> /IOB_13B
- J2 pad 11: /IOB_13B -> /IOB_16A
- J2 pad 12: /IOB_8A -> /IOB_18A
- J2 pad 13: /IOB_9B -> /IOB_20A
- J2 pad 14: /IOB_6A -> /IOB_22A
- J2 pad 7: /IOB_22A -> /IOB_6A
- J2 pad 8: /IOB_20A -> /IOB_9B
- J2 pad 9: /IOB_18A -> /IOB_8A
- J3 pad 10: /IOT_41A -> /IOT_42B
- J3 pad 11: /IOT_42B -> /IOT_41A
- J3 pad 12: /IOT_43A -> /IOT_38B
- J3 pad 13: /IOT_44B -> /IOT_39A
- J3 pad 14: /IOT_48B -> /IOT_36B
- J3 pad 7: /IOT_36B -> /IOT_48B
- J3 pad 8: /IOT_39A -> /IOT_44B
- J3 pad 9: /IOT_38B -> /IOT_43A
- Q1 pad 1: /IOB_22A -> /IOB_6A
- Q10 pad 1: /IOT_42B -> /IOT_41A
- Q11 pad 1: /IOB_8A -> /IOB_18A
- Q12 pad 1: /IOT_43A -> /IOT_38B
- Q13 pad 1: /IOB_9B -> /IOB_20A
- Q14 pad 1: /IOT_44B -> /IOT_39A
- Q15 pad 1: /IOB_6A -> /IOB_22A
- Q16 pad 1: /IOT_48B -> /IOT_36B
- Q2 pad 1: /IOT_36B -> /IOT_48B
- Q3 pad 1: /IOB_20A -> /IOB_9B
- Q4 pad 1: /IOT_39A -> /IOT_44B
- Q5 pad 1: /IOB_18A -> /IOB_8A
- Q6 pad 1: /IOT_38B -> /IOT_43A
- Q7 pad 1: /IOB_16A -> /IOB_13B
- Q8 pad 1: /IOT_41A -> /IOT_42B
- Q9 pad 1: /IOB_13B -> /IOB_16A
- R16 pad 1: /IOB_22A -> /IOB_6A
- R17 pad 1: /IOT_36B -> /IOT_48B
- R20 pad 1: /IOB_20A -> /IOB_9B
- R21 pad 1: /IOT_39A -> /IOT_44B
- R32 pad 1: /IOB_18A -> /IOB_8A
- R33 pad 1: /IOT_38B -> /IOT_43A
- R36 pad 1: /IOB_16A -> /IOB_13B
- R37 pad 1: /IOT_41A -> /IOT_42B
- R40 pad 1: /IOB_13B -> /IOB_16A
- R41 pad 1: /IOT_42B -> /IOT_41A
- R44 pad 1: /IOB_8A -> /IOB_18A
- R45 pad 1: /IOT_43A -> /IOT_38B
- R48 pad 1: /IOB_9B -> /IOB_20A
- R49 pad 1: /IOT_44B -> /IOT_39A
- R52 pad 1: /IOB_6A -> /IOB_22A
- R53 pad 1: /IOT_48B -> /IOT_36B
Routing:
- net /RGB2: track 0.95 -> 25.4 mm, vias 1 -> 2
- net Net-(IC4-CH1): track 3.50 -> 27.7 mm, vias 1 -> 3
- net /RGB0: track 0.95 -> 24.5 mm, vias 1 -> 2
- net Net-(IC4-CH0): track 4.04 -> 25.4 mm, vias 1 -> 2
- net /IOB_22A: track 28.8 -> 7.86 mm, vias 3 -> 1
- net /IOT_36B: track 31.3 -> 10.4 mm, vias 3 -> 2
- net /IOT_48B: track 18.2 -> 38.9 mm
- net /RGB1: track 0.85 -> 21.3 mm, vias 1 -> 2
- net Net-(IC4-CH3): track 3.67 -> 23.9 mm, vias 1 -> 4
- net /IOB_6A: track 15.3 -> 32.4 mm
- net /IOT_39A: track 28.9 -> 12.7 mm, vias 3 -> 2
- net /IOB_20A: track 26.4 -> 11.3 mm, vias 3 -> 2
- net Net-(IC4-CH2): track 3.36 -> 18.0 mm, vias 1 -> 2
- net /IOT_44B: track 22.6 -> 35.7 mm, vias 3 -> 2
- net /IOB_9B: track 16.3 -> 29.2 mm
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
Commit message: Finished DRAFT wiring (NB3 Hindbrain)
Connections:
- IC1 pad 65: unconnected-(IC1-TP-Pad65) -> GND
- IC2 pad 13: /IOB_24A -> unconnected-(IC2-IOB_24A-Pad13)
- IC2 pad 23: unconnected-(IC2-IOT_37A-Pad23) -> /IOT_37A
- IC2 pad V49_1: (no net) -> GND
- IC2 pad V49_10: (no net) -> GND
- IC2 pad V49_11: (no net) -> GND
- IC2 pad V49_12: (no net) -> GND
- IC2 pad V49_13: (no net) -> GND
- IC2 pad V49_14: (no net) -> GND
- IC2 pad V49_15: (no net) -> GND
- IC2 pad V49_16: (no net) -> GND
- IC2 pad V49_17: (no net) -> GND
- IC2 pad V49_18: (no net) -> GND
- IC2 pad V49_19: (no net) -> GND
- IC2 pad V49_2: (no net) -> GND
- IC2 pad V49_20: (no net) -> GND
- IC2 pad V49_21: (no net) -> GND
- IC2 pad V49_3: (no net) -> GND
- IC2 pad V49_4: (no net) -> GND
- IC2 pad V49_5: (no net) -> GND
- IC2 pad V49_6: (no net) -> GND
- IC2 pad V49_7: (no net) -> GND
- IC2 pad V49_8: (no net) -> GND
- IC2 pad V49_9: (no net) -> GND
- IC4 pad 10: /IOB_31B -> /IOB_29B
- IC4 pad 11: /IOB_24A -> /IOB_31B
- IC4 pad 8: /IOB_23B -> /IOT_37A
- IC4 pad 9: /IOB_29B -> /IOB_23B
- J1 pad 10: (no net) -> GND
- J1 pad 11: (no net) -> GND
Routing:
- net /FPGA_SCLK: track 13.8 -> 65.8 mm
- net /FLASH_MISO: track 9.20 -> 56.7 mm
- net /FPGA_CS: track 11.1 -> 58.5 mm
- net /FLASH_MOSI: track 11.8 -> 59.1 mm
- net /CRESET: track 20.0 -> 54.9 mm, vias 2 -> 3
- net /CDONE: track 2.90 -> 36.6 mm
- net GND: track 99.2 -> 117.4 mm
- net /IOB_3B_G6: track 1.06 -> 17.1 mm, vias 1 -> 2
- net /IOB_24A: track 11.9 -> 0.00 mm, vias 1 -> 0
- net /IOB_25B_G3: track 0.86 -> 8.86 mm, vias 1 -> 2
- net +3V3: track 183.0 -> 186.4 mm
- net /IOT_37A: track 0.00 -> 2.25 mm, vias 0 -> 1
- net /IOB_23B: track 2.12 -> 4.16 mm, vias 1 -> 2
- net /RGB1: track 21.3 -> 22.6 mm
- net /RGB2: track 25.4 -> 26.7 mm
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