File: boxes/fpgas/NB3_hindbrain/NB3_hindbrain.kicad_pcb (KiCad board)
At the start: 4 copper layers, 57 x 22.5 mm, 147 parts, among them IC1 FT2232HQ, IC2 FPGA_ICE40UP5K-SG48I, IC3 NOR_Flash_W25Q32JVSSIQ, IC4 ADC_MCP3004-I-SL, IC5 MCP4812-E_SN, J1 MicroUSB_10103594-0001LF, J2 Conn_01x20_Pin, J3 Conn_01x20_Pin, Q1 RUM001L02T2CL, Q10 RUM001L02T2CL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

Commit message: NB3 Hindbrain prototype (sent to fab)
Parts:
- removed LED1: CLMVC-FKA-CLBDGL7LBB79353, NB3_hindbrain:RGB_CLMVC-FKA-CLBDGL7LBB79353
- added RGB1: CLMVC-FKA-CLBDGL7LBB79353, NB3_hindbrain:RGB_CLMVC-FKA-CLBDGL7LBB79353, F.Cu at (111.6, 80.0)
- D1: value LED -> LED (W)
- D10, D12, D14, D16, D18, D2, D20, D6, D8: value LED -> LED (B)
- D11, D13, D15, D17, D19, D21, D3, D7, D9: value LED -> LED (R)
- R18, R19, R30, R31, R34, R35, R38, R39, R42, R43, R46, R47, R50, R51, R54, R55, R8, R9: value 680 -> 330
Routing:
- net GND: track 117.4 -> 153.3 mm
Other:
- board text added: "locked"
- board text removed: "3v3"
- board text removed: "5V"
- board text removed: "A0"
- board text removed: "A1"
- board text removed: "A2"
- board text removed: "A3"
- board text removed: "CK"
- board text removed: "CS"
- board text removed: "D0"
- board text removed: "D1"
- board text removed: "For Research and Education ONLY"
- board text removed: "Gnd"
- board text removed: "Hz"
- board text removed: "L0"
- board text removed: "L1"
- board text removed: "L2"
- board text removed: "L3"
- board text removed: "L4"
- board text removed: "L5"
- board text removed: "L6"
- board text removed: "L7"
- board text removed: "LG"
- board text removed: "NB3 Hindbrain"
- board text removed: "PWR"
- board text removed: "R0"
- board text removed: "R1"
- board text removed: "R2"
- board text removed: "R3"
- board text removed: "R4"
- board text removed: "R5"
- board text removed: "R6"
- board text removed: "R7"
- board text removed: "RG"
- board text removed: "Rst"
- board text removed: "Rx"
- board text removed: "SI"
- board text removed: "SO"
- board text removed: "Tx"
- board text removed: "rev 0.0.1"
