File: boxes/fpgas/NB3_hindbrain/NB3_hindbrain.kicad_sch (KiCad schematic)
At the start: 147 parts, among them IC1 FT2232HQ, IC2 FPGA_ICE40UP5K-SG48I, IC3 NOR_Flash_W25Q32JVSSIQ, IC4 ADC_MCP3004-I-SL, IC5 MCP4812-E_SN, J1 MicroUSB_10103594-0001LF, J2 Conn_01x20_Pin, J3 Conn_01x20_Pin, Q1 RUM001L02T2CL, Q10 RUM001L02T2CL, Q11 RUM001L02T2CL, Q12 RUM001L02T2CL, Q13 RUM001L02T2CL, Q14 RUM001L02T2CL, Q15 RUM001L02T2CL, Q16 RUM001L02T2CL, Q2 RUM001L02T2CL, Q3 RUM001L02T2CL, Q4 RUM001L02T2CL, Q5 RUM001L02T2CL, Q6 RUM001L02T2CL, Q7 RUM001L02T2CL, Q8 RUM001L02T2CL, Q9 RUM001L02T2CL, U1 EEPROM_93LC56BT-I-OT, Y1 Osc_12MHz_ECS-2520MV-120-BN-TR

Commit message: Wiring progress...
Connections:
- net IOB_0A: now also IC5.3 (SCK); no longer IC4.9 (DIN)
- net IOB_13B: now also J2.10 (Pin_10), Q7.1 (G), R36.1; no longer J2.11 (Pin_11), Q9.1 (G), R40.1
- net IOB_16A: now also J2.11 (Pin_11), Q9.1 (G), R40.1; no longer J2.10 (Pin_10), Q7.1 (G), R36.1
- net IOB_18A: now also J2.12 (Pin_12), Q11.1 (G), R44.1; no longer J2.9 (Pin_9), Q5.1 (G), R32.1
- net IOB_20A: now also J2.13 (Pin_13), Q13.1 (G), R48.1; no longer J2.8 (Pin_8), Q3.1 (G), R20.1
- net IOB_22A: now also J2.14 (Pin_14), Q15.1 (G), R52.1; no longer J2.7 (Pin_7), Q1.1 (G), R16.1
- net IOB_23B: now also IC4.8 (~{CS}/SHDN); no longer IC5.5 (~{LDAC})
- net IOB_24A: now also IC4.11 (CLK); no longer IC5.2 (~{CS})
- net IOB_29B: now also IC4.9 (DIN); no longer IC5.4 (SDI)
- net IOB_2A: now also IC5.2 (~{CS}); no longer IC4.10 (DOUT)
- net IOB_31B: now also IC4.10 (DOUT); no longer IC5.3 (SCK)
- net IOB_4A: now also IC5.5 (~{LDAC}); no longer IC4.11 (CLK)
- net IOB_5B: now also IC5.4 (SDI); no longer IC4.8 (~{CS}/SHDN)
- net IOB_6A: now also J2.7 (Pin_7), Q1.1 (G), R16.1; no longer J2.14 (Pin_14), Q15.1 (G), R52.1
- net IOB_8A: now also J2.9 (Pin_9), Q5.1 (G), R32.1; no longer J2.12 (Pin_12), Q11.1 (G), R44.1
- net IOB_9B: now also J2.8 (Pin_8), Q3.1 (G), R20.1; no longer J2.13 (Pin_13), Q13.1 (G), R48.1
- net IOT_36B: now also J3.14 (Pin_14), Q16.1 (G), R53.1; no longer J3.7 (Pin_7), Q2.1 (G), R17.1
- net IOT_38B: now also J3.12 (Pin_12), Q12.1 (G), R45.1; no longer J3.9 (Pin_9), Q6.1 (G), R33.1
- net IOT_39A: now also J3.13 (Pin_13), Q14.1 (G), R49.1; no longer J3.8 (Pin_8), Q4.1 (G), R21.1
- net IOT_41A: now also J3.11 (Pin_11), Q10.1 (G), R41.1; no longer J3.10 (Pin_10), Q8.1 (G), R37.1
- net IOT_42B: now also J3.10 (Pin_10), Q8.1 (G), R37.1; no longer J3.11 (Pin_11), Q10.1 (G), R41.1
- net IOT_43A: now also J3.9 (Pin_9), Q6.1 (G), R33.1; no longer J3.12 (Pin_12), Q12.1 (G), R45.1
- net IOT_44B: now also J3.8 (Pin_8), Q4.1 (G), R21.1; no longer J3.13 (Pin_13), Q14.1 (G), R49.1
- net IOT_48B: now also J3.7 (Pin_7), Q2.1 (G), R17.1; no longer J3.14 (Pin_14), Q16.1 (G), R53.1

Commit message: Finished DRAFT wiring (NB3 Hindbrain)
Connections:
- net GND: now also IC1.65 (TP), IC2.V49_1 (SH), IC2.V49_10 (SH), IC2.V49_11 (SH), IC2.V49_12 (SH), IC2.V49_13 (SH), IC2.V49_14 (SH), IC2.V49_15 (SH), IC2.V49_16 (SH), IC2.V49_17 (SH), IC2.V49_18 (SH), IC2.V49_19 (SH), IC2.V49_2 (SH), IC2.V49_20 (SH), IC2.V49_21 (SH), IC2.V49_3 (SH), IC2.V49_4 (SH), IC2.V49_5 (SH), IC2.V49_6 (SH), IC2.V49_7 (SH), IC2.V49_8 (SH), IC2.V49_9 (SH), J1.10 (SH), J1.11 (SH)
- net IOB_23B: now also IC4.9 (DIN); no longer IC4.8 (~{CS}/SHDN)
- net IOB_29B: now also IC4.10 (DOUT); no longer IC4.9 (DIN)
- net IOB_31B: now also IC4.11 (CLK); no longer IC4.10 (DOUT)
- net IOT_37A: now reaches IC2.23 (IOT_37A)
- net IOT_37A: now also IC4.8 (~{CS}/SHDN)
- net IOB_24A: no longer names the net of IC2.13 (IOB_24A)
- net IOB_24A: no longer IC4.11 (CLK)
- no-connect marks 34 -> 33
Changed lines of the file:
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@@
   (title_block
     (title "NB3 Hindbrain (FPGA) Board")
-    (date "2023-08-25")
+    (date "2023-08-29")
     (rev "0.0.1")
     (company "Voight-Kampff")
@@
   (junction (at 13.97 49.53) (diameter 0.9144) (color 0 0 0 0)
   )
+  (junction (at 36.83 52.07) (diameter 0) (color 0 0 0 0)
+  )
   (junction (at 13.97 52.07) (diameter 0.9144) (color 0 0 0 0)
   )
@@
   (junction (at 62.865 142.875) (diameter 0.9144) (color 0 0 0 0)
   )
+  (junction (at 76.835 48.26) (diameter 0) (color 0 0 0 0)
+  )
   (junction (at 25.4 57.15) (diameter 0.9144) (color 0 0 0 0)
   )
@@
   (junction (at 254.635 189.23) (diameter 0.9144) (color 0 0 0 0)
   )
+  (junction (at 238.76 78.74) (diameter 0) (color 0 0 0 0)
+  )
   (junction (at 227.33 114.3) (diameter 0.9144) (color 0 0 0 0)
   )
@@
   (no_connect (at 132.715 53.34))
   (no_connect (at 242.57 185.42))
-  (no_connect (at 212.09 106.68))
   (no_connect (at 104.775 27.94))
+  (no_connect (at 186.69 106.68))
   (no_connect (at 117.475 27.94))
   (no_connect (at 114.935 27.94))
@@
   (no_connect (at 132.715 68.58))
   (no_connect (at 36.83 44.45))
-  (no_connect (at 84.455 27.94))
   (no_connect (at 201.93 25.4))
   (no_connect (at 310.515 153.035))
@@
     (stroke (width 0) (type default))
   )
+  (wire (pts (xy 222.25 87.63) (xy 238.76 87.63))
+    (stroke (width 0) (type default))
+  )
   (polyline (pts (xy 255.27 69.85) (xy 387.35 69.85))
     (stroke (width 0.5) (type solid))
@@
     (stroke (width 0) (type solid))
   )
-  (wire (pts (xy 36.83 57.15) (xy 36.83 46.99))
+  (wire (pts (xy 36.83 57.15) (xy 36.83 52.07))
     (stroke (width 0) (type solid))
   )
@@
     (stroke (width 0) (type default))
   )
+  (wire (pts (xy 34.29 52.07) (xy 36.83 52.07))
+    (stroke (width 0) (type default))
+  )
   (wire (pts (xy 64.77 192.405) (xy 64.77 189.865))
     (stroke (width 0) (type solid))
@@
     (stroke (width 0) (type dash))
   )
+  (wire (pts (xy 36.83 52.07) (xy 36.83 46.99))
+    (stroke (width 0) (type solid))
+  )
   (wire (pts (xy 306.705 137.16) (xy 306.705 142.875))
     (stroke (width 0) (type default))
@@
     (stroke (width 0) (type default))
   )
+  (wire (pts (xy 238.76 87.63) (xy 238.76 78.74))
+    (stroke (width 0) (type default))
+  )
   (wire (pts (xy 21.59 76.2) (xy 29.845 76.2))
     (stroke (width 0) (type default))
@@
     (stroke (width 0) (type default))
   )
+  (wire (pts (xy 76.835 27.94) (xy 76.835 48.26))
+    (stroke (width 0) (type default))
+  )
   (wire (pts (xy 139.7 137.795) (xy 139.7 140.335))
     (stroke (width 0) (type default))
@@
     (stroke (width 0) (type default))
   )
+  (wire (pts (xy 84.455 27.94) (xy 76.835 27.94))
+    (stroke (width 0) (type default))
+  )
   (wire (pts (xy 13.97 34.29) (xy 13.97 36.83))
     (stroke (width 0) (type solid))
@@
     (effects (font (size 1.27 1.27)) (justify left bottom))
   )
-  (text "ICE40 UltraPlus FPGA\n(ICE40UP5K-SG48I)" (at 254 20.32 0)
+  (text "ICE40 UltraPlus FPGA\n(ICE40UP5K-SG48I)" (at 252.476 20.32 0)
     (effects (font (size 2 2) (thickness 0.4) bold) (justify right bottom))
   )
@@
     (effects (font (size 1.27 1.27)) (justify right bottom))
   )
-  (label "IOB_31B" (at 343.535 150.495 0) (fields_autoplaced)
+  (label "IOB_31B" (at 343.535 147.955 0) (fields_autoplaced)
     (effects (font (size 1.27 1.27)) (justify left bottom))
   )
@@
     (effects (font (size 1.27 1.27)) (justify right bottom))
   )
-  (label "IOB_24A" (at 343.535 147.955 0) (fields_autoplaced)
-    (effects (font (size 1.27 1.27)) (justify left bottom))
-  )
   (label "CLK_12MHz" (at 266.7 181.61 0) (fields_autoplaced)
     (effects (font (size 1.27 1.27)) (justify left bottom))
@@
     (effects (font (size 1.27 1.27)) (justify right bottom))
   )
-  (label "IOB_29B" (at 343.535 153.035 0) (fields_autoplaced)
+  (label "IOB_29B" (at 343.535 150.495 0) (fields_autoplaced)
     (effects (font (size 1.27 1.27)) (justify left bottom))
   )
@@
     (effects (font (size 1.27 1.27)) (justify right bottom))
   )
-  (label "IOB_24A" (at 186.69 106.68 270) (fields_autoplaced)
-    (effects (font (size 1.27 1.27)) (justify right bottom))
-  )
   (label "FPGA_SCLK" (at 191.77 106.68 270) (fields_autoplaced)
     (effects (font (size 1.27 1.27)) (justify right bottom))
@@
     (effects (font (size 1.27 1.27)) (justify left bottom))
   )
+  (label "IOT_37A" (at 343.535 155.575 0) (fields_autoplaced)
+    (effects (font (size 1.27 1.27)) (justify left bottom))
+  )
   (label "USB_5V" (at 264.16 102.235 270) (fields_autoplaced)
     (effects (font (size 1.27 1.27)) (justify right bottom))
@@
     (effects (font (size 1.27 1.27)) (justify right bottom))
   )
-  (label "IOB_23B" (at 343.535 155.575 0) (fields_autoplaced)
+  (label "IOB_23B" (at 343.535 153.035 0) (fields_autoplaced)
     (effects (font (size 1.27 1.27)) (justify left bottom))
   )
@@
     (effects (font (size 1.27 1.27)) (justify right bottom))
   )
+  (label "IOT_37A" (at 212.09 106.68 270) (fields_autoplaced)
+    (effects (font (size 1.27 1.27)) (justify right bottom))
+  )
   (label "CLK_12MHz" (at 269.24 88.265 90) (fields_autoplaced)
     (effects (font (size 1.27 1.27)) (justify left bottom))
@@
     (pin "S1")
     (pin "S2")
+    (pin "10")
+    (pin "11")
     (instances
       (project "NB3_hindbrain"
@@
     (pin "8")
     (pin "9")
+    (pin "V49_1")
+    (pin "V49_10")
+    (pin "V49_11")
+    (pin "V49_12")
+    (pin "V49_13")
+    (pin "V49_14")
+    (pin "V49_15")
+    (pin "V49_16")
+    (pin "V49_17")
+    (pin "V49_18")
+    (pin "V49_19")
+    (pin "V49_2")
+    (pin "V49_20")
+    (pin "V49_21")
+    (pin "V49_3")
+    (pin "V49_4")
+    (pin "V49_5")
+    (pin "V49_6")
+    (pin "V49_7")
+    (pin "V49_8")
+    (pin "V49_9")
     (instances
       (project "NB3_hindbrain"
@@
     )
   )
-  (symbol (lib_id "NB3_hindbrain:Logo_VK") (at 140.97 108.585 0) (unit 1)
+  (symbol (lib_id "NB3_hindbrain:Logo_VK") (at 139.7 106.68 0) (unit 1)
     (in_bom yes) (on_board yes) (dnp no) (fields_autoplaced)
-    (property "Reference" "G2" (at 140.97 122.555 0)
+    (property "Reference" "G2" (at 139.7 120.65 0)
       (effects (font (size 1.27 1.27)) hide)
     )
-    (property "Value" "Logo_VK" (at 140.97 94.615 0)
+    (property "Value" "Logo_VK" (at 139.7 92.71 0)
       (effects (font (size 1.27 1.27)) hide)
     )
-    (property "Footprint" "NB3_hindbrain:Logo_VK_5mm" (at 140.97 108.585 0)
+    (property "Footprint" "NB3_hindbrain:Logo_VK_5mm" (at 139.7 106.68 0)
       (effects (font (size 1.27 1.27)) hide)
     )
-    (property "Datasheet" "" (at 140.97 108.585 0)
+    (property "Datasheet" "" (at 139.7 106.68 0)
       (effects (font (size 1.27 1.27)) hide)
     )

Commit message: NB3 Hindbrain prototype (sent to fab)
Parts:
- D1: value LED -> LED (W)
- D10, D12, D14, D16, D18, D2, D20, D6, D8: value LED -> LED (B)
- D11, D13, D15, D17, D19, D21, D3, D7, D9: value LED -> LED (R)
- R18, R19, R30, R31, R34, R35, R38, R39, R42, R43, R46, R47, R50, R51, R54, R55, R8, R9: value 680 -> 330
- renumbered LED1 to RGB1
Changed lines of the file:
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@@
     (stroke (width 0) (type default))
   )
-  (text "12 MHz Clock" (at 264.795 172.72 0)
+  (text "12 MHz Clock" (at 264.795 172.085 0)
     (effects (font (size 2 2) (thickness 0.4) bold) (justify right bottom))
   )
@@
       (effects (font (size 1.27 1.27)))
     )
-    (property "Value" "680" (at 288.925 48.26 90)
+    (property "Value" "330" (at 288.925 48.26 90)
       (effects (font (size 1 1)))
     )
@@
       (effects (font (size 1.27 1.27)))
     )
-    (property "Value" "680" (at 377.825 48.26 90)
+    (property "Value" "330" (at 377.825 48.26 90)
       (effects (font (size 1 1)))
     )
@@
       (effects (font (size 0.5 0.5)))
     )
-    (property "Value" "LED" (at 310.7055 40.64 90)
+    (property "Value" "LED (R)" (at 310.7055 40.64 90)
       (effects (font (size 1.27 1.27)) hide)
     )
@@
       (effects (font (size 1.27 1.27)))
     )
-    (property "Value" "680" (at 327.025 48.26 90)
+    (property "Value" "330" (at 327.025 48.26 90)
       (effects (font (size 1 1)))
     )
@@
       (effects (font (size 1.27 1.27)))
     )
-    (property "Value" "680" (at 109.22 189.23 90)
+    (property "Value" "330" (at 109.22 189.23 90)
       (effects (font (size 1.27 1.27)))
     )
@@
       (effects (font (size 0.5 0.5)))
     )
-    (property "Value" "LED" (at 298.0055 40.64 90)
+    (property "Value" "LED (R)" (at 298.0055 40.64 90)
       (effects (font (size 1.27 1.27)) hide)
     )
@@
       (effects (font (size 0.5 0.5)))
     )
-    (property "Value" "LED" (at 298.0055 13.97 90)
+    (property "Value" "LED (B)" (at 298.0055 13.97 90)
       (effects (font (size 1.27 1.27)) hide)
     )
@@
       (effects (font (size 1.27 1.27)))
     )
-    (property "Value" "680" (at 301.625 48.26 90)
+    (property "Value" "330" (at 301.625 48.26 90)
       (effects (font (size 1 1)))
     )
@@
       (effects (font (size 0.5 0.5)))
     )
-    (property "Value" "LED" (at 348.8055 13.97 90)
+    (property "Value" "LED (B)" (at 348.8055 13.97 90)
       (effects (font (size 1.27 1.27)) hide)
     )
@@
       (effects (font (size 1.27 1.27)))
     )
-    (property "Value" "680" (at 377.825 21.59 90)
+    (property "Value" "330" (at 377.825 21.59 90)
       (effects (font (size 1 1)))
     )
@@
       (effects (font (size 0.5 0.5)))
     )
-    (property "Value" "LED" (at 285.3055 40.64 90)
+    (property "Value" "LED (R)" (at 285.3055 40.64 90)
       (effects (font (size 1.27 1.27)) hide)
     )
@@
       (effects (font (size 0.5 0.5)))
     )
-    (property "Value" "LED" (at 310.7055 13.97 90)
+    (property "Value" "LED (B)" (at 310.7055 13.97 90)
       (effects (font (size 1.27 1.27)) hide)
     )
@@
       (effects (font (size 1.27 1.27)))
     )
-    (property "Value" "680" (at 339.725 21.59 90)
+    (property "Value" "330" (at 339.725 21.59 90)
       (effects (font (size 1 1)))
     )
@@
       (effects (font (size 1.27 1.27)))
     )
-    (property "Value" "680" (at 352.425 48.26 90)
+    (property "Value" "330" (at 352.425 48.26 90)
       (effects (font (size 1 1)))
     )
@@
   (symbol (lib_id "NB3_hindbrain:RGB_CLMVC-FKA-CLBDGL7LBB79353") (at 143.51 180.34 0) (unit 1)
     (in_bom yes) (on_board yes) (dnp no)
-    (property "Reference" "LED1" (at 147.32 178.435 0)
+    (property "Reference" "RGB1" (at 147.32 178.435 0)
       (effects (font (size 1.27 1.27)))
     )
@@
       (project "NB3_hindbrain"
         (path "/c49eb9c2-071f-42f1-813b-8f9aeee9d910"
-          (reference "LED1") (unit 1)
+          (reference "RGB1") (unit 1)
         )
       )
@@
       (effects (font (size 1.27 1.27)))
     )
-    (property "Value" "680" (at 365.125 21.59 90)
+    (property "Value" "330" (at 365.125 21.59 90)
       (effects (font (size 1 1)))
     )
@@
       (effects (font (size 1.27 1.27)))
     )
-    (property "Value" "680" (at 352.425 21.59 90)
+    (property "Value" "330" (at 352.425 21.59 90)
       (effects (font (size 1 1)))
     )
@@
       (effects (font (size 1.27 1.27)))
     )
-    (property "Value" "680" (at 288.925 21.59 90)
+    (property "Value" "330" (at 288.925 21.59 90)
       (effects (font (size 1 1)))
     )
@@
       (effects (font (size 1.27 1.27)))
     )
-    (property "Value" "680" (at 314.325 21.59 90)
+    (property "Value" "330" (at 314.325 21.59 90)
       (effects (font (size 1 1)))
     )
@@
       (effects (font (size 0.5 0.5)))
     )
-    (property "Value" "LED" (at 285.3055 13.97 90)
+    (property "Value" "LED (B)" (at 285.3055 13.97 90)
       (effects (font (size 1.27 1.27)) hide)
     )
@@
       (effects (font (size 1.27 1.27)))
     )
-    (property "Value" "680" (at 119.38 189.23 90)
+    (property "Value" "330" (at 119.38 189.23 90)
       (effects (font (size 1.27 1.27)))
     )
@@
       (effects (font (size 1.27 1.27)))
     )
-    (property "Value" "LED" (at 108.585 181.61 0)
+    (property "Value" "LED (B)" (at 108.585 181.61 0)
       (effects (font (size 1.27 1.27)))
     )
@@
       (effects (font (size 1.27 1.27)))
     )
-    (property "Value" "680" (at 365.125 48.26 90)
+    (property "Value" "330" (at 365.125 48.26 90)
       (effects (font (size 1 1)))
     )
@@
       (effects (font (size 0.5 0.5)))
     )
-    (property "Value" "LED" (at 323.4055 40.64 90)
+    (property "Value" "LED (R)" (at 323.4055 40.64 90)
       (effects (font (size 1.27 1.27)) hide)
     )
@@
       (effects (font (size 0.5 0.5)))
     )
-    (property "Value" "LED" (at 361.5055 13.97 90)
+    (property "Value" "LED (B)" (at 361.5055 13.97 90)
       (effects (font (size 1.27 1.27)) hide)
     )
@@
       (effects (font (size 0.5 0.5)))
     )
-    (property "Value" "LED" (at 336.1055 13.97 90)
+    (property "Value" "LED (B)" (at 336.1055 13.97 90)
       (effects (font (size 1.27 1.27)) hide)
     )
@@
       (effects (font (size 1.27 1.27)))
     )
-    (property "Value" "680" (at 301.625 21.59 90)
+    (property "Value" "330" (at 301.625 21.59 90)
       (effects (font (size 1 1)))
     )
@@
       (effects (font (size 0.5 0.5)))
     )
-    (property "Value" "LED" (at 348.8055 40.64 90)
+    (property "Value" "LED (R)" (at 348.8055 40.64 90)
       (effects (font (size 1.27 1.27)) hide)
     )
@@
       (effects (font (size 0.5 0.5)))
     )
-    (property "Value" "LED" (at 374.2055 13.97 90)
+    (property "Value" "LED (B)" (at 374.2055 13.97 90)
       (effects (font (size 1.27 1.27)) hide)
     )
@@
       (effects (font (size 0.5 0.5)))
     )
-    (property "Value" "LED" (at 323.4055 13.97 90)
+    (property "Value" "LED (B)" (at 323.4055 13.97 90)
       (effects (font (size 1.27 1.27)) hide)
     )
@@
       (effects (font (size 1.27 1.27)))
     )
-    (property "Value" "680" (at 339.725 48.26 90)
+    (property "Value" "330" (at 339.725 48.26 90)
       (effects (font (size 1 1)))
     )
@@
       (effects (font (size 0.5 0.5)))
     )
-    (property "Value" "LED" (at 374.2055 40.64 90)
+    (property "Value" "LED (R)" (at 374.2055 40.64 90)
       (effects (font (size 1.27 1.27)) hide)
     )
@@
       (effects (font (size 1.27 1.27)))
     )
-    (property "Value" "680" (at 327.025 21.59 90)
+    (property "Value" "330" (at 327.025 21.59 90)
       (effects (font (size 1 1)))
     )
@@
       (effects (font (size 0.5 0.5)))
     )
-    (property "Value" "LED" (at 361.5055 40.64 90)
+    (property "Value" "LED (R)" (at 361.5055 40.64 90)
       (effects (font (size 1.27 1.27)) hide)
     )
@@
       (effects (font (size 1.27 1.27)))
     )
-    (property "Value" "LED" (at 89.535 181.61 0)
+    (property "Value" "LED (W)" (at 89.535 181.61 0)
       (effects (font (size 1.27 1.27)))
     )
@@
       (effects (font (size 0.5 0.5)))
     )
-    (property "Value" "LED" (at 336.1055 40.64 90)
+    (property "Value" "LED (R)" (at 336.1055 40.64 90)
       (effects (font (size 1.27 1.27)) hide)
     )
@@
       (effects (font (size 1.27 1.27)))
     )
-    (property "Value" "680" (at 314.325 48.26 90)
+    (property "Value" "330" (at 314.325 48.26 90)
       (effects (font (size 1 1)))
     )
@@
       (effects (font (size 1.27 1.27)))
     )
-    (property "Value" "LED" (at 118.745 181.61 0)
+    (property "Value" "LED (R)" (at 118.745 181.61 0)
       (effects (font (size 1.27 1.27)))
     )
