File: boxes/electrons/NB3_body/NB3_body.kicad_pcb (KiCad board)
At the start: 2 copper layers, 200 x 199.5 mm, 41 parts, among them J1 Conn_02x05_Counter_Clockwise, J10 JST SH 4-way Socket, J12 Conn_02x03_Top_Bottom, J13 Conn_02x03_Top_Bottom, J14 Conn_02x05_Counter_Clockwise, J15 Conn_02x05_Counter_Clockwise, J2 Conn_02x05_Counter_Clockwise, J3 Conn_02x05_Counter_Clockwise, J4 Conn_02x05_Counter_Clockwise, J5 Conn_02x05_Counter_Clockwise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

Commit message: Update NB3_Body (fix right ear orientation)
Parts:
- turned J8 to 0 degrees
Routing:
- net /SCK: track 274.9 -> 281.2 mm
- net +3V3: track 265.6 -> 271.5 mm
- net /SDI: track 246.5 -> 250.9 mm
- net /WS: track 310.4 -> 314.7 mm, vias 4 -> 5
Other:
- board text added: "0v 0v 5v 5v"
- board text added: "0v WS SI 0v 0v 3.3 CK"
- board text added: "3.3"
- board text added: "3.3 WS SI 0v 0v 3.3 CK"
- board text added: "GA"
- board text added: "GA WS SO 0v 0v 5v CK"
- board text added: "NB3_body Rev 0.0.5 For Research and Education ONLY"
- board text added: "SO SI"
- board text added: "WS CK"
- board text removed: "0v 0v rA rB rC 5v 5v lA lB lC"
- board text removed: "NB3_body Rev 0.0.4 For Research and Education ONLY"
