File: power/NB3_power/NB3_power.kicad_pcb (KiCad board)
At the start: 2 copper layers, 51 x 45 mm, 34 parts, among them J1 Barrel_Jack_PJ-036AH-SMT-TR, J2 Connector_S4B-PH-SM4-TB(LF)(S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, SW1 SW_SPDT, U1 Voltage_Regulator_AP64501

Commit message: Update PCBs (body, ear, mouth, and power)
Parts:
- removed G***: LOGO, NB3_power:Logo_VK_15mm
- added J3: Conn_01x02_Pin, Connector_PinHeader_2.54mm:PinHeader_1x02_P2.54mm_Horizontal, F.Cu at (152.8, 119.4)
Routing:
- net +12V: track 42.8 -> 50.5 mm, vias 4 -> 5
Other:
- board text added: "Input [+V +V]"
- board text added: "NB3_power Rev 0.0.5"
- board text removed: "NB3_power Rev 0.0.4"
